File: Proyecto Final/Circuitos del kicad/Proyecto V1/_autosave-Proyecto V1.kicad_pcb (KiCad board)
At the start: 2 copper layers, 14 parts, among them J1 12v, J2 I2C + LCD, J3 DS1307, SW1 SW_Push, SW2 SW_Push, SW3 SW_Push, SW4 SW_Push, U1 LM7805_TO220, U2 DS18B20, U3 ATmega328P-P

Commit message: save kicad
Parts:
- --------1: value Sensor nivel -> lvl_sens
- moved J3 5.68 mm to (175.3, 55.9), turned to 0 degrees
- turned J2 to 0 degrees
Routing:
- net +5V: track 49.8 -> 70.7 mm
- net GND: track 183.5 -> 201.0 mm
- net Net-(J2-PadSDA): track 0.00 -> 10.8 mm
- net Net-(J2-PadSCL): track 0.00 -> 10.2 mm
- net Net-(U3-Pad7): track 3.18 -> 0.64 mm
