File: Proyecto Final/Circuitos del kicad/Proyecto V1/Proyecto V1.kicad_pcb (KiCad board)
At the start: 2 copper layers, 15 parts, among them J1 12v, J2 I2C + LCD, J3 DS1307, J4 5v, SW1 SW_Push, SW2 SW_Push, SW3 SW_Push, SW4 SW_Push, U1 LM7805_TO220, U2 DS18B20, U3 ATmega328P-P

Commit message: save kicad
Parts:
- removed J4: 5v, TerminalBlock:TerminalBlock_bornier-2_P5.08mm
- --------1: value Sensor nivel -> lvl_sens
- moved J1 41.7 mm to (165.1, 119.1), turned to 180 degrees
- moved U1 41.0 mm to (160.0, 106.4), turned to 0 degrees
- moved SW4 15.2 mm to (145.9, 99.0), turned to 180 degrees
- moved SW3 12.9 mm to (145.9, 83.8), turned to 180 degrees
- moved SW2 10.8 mm to (145.9, 68.5), turned to 180 degrees
- moved SW1 8.80 mm to (145.9, 53.3), turned to 180 degrees
- moved J3 1.38 mm to (175.3, 55.9)
- moved J2 1.38 mm to (170.2, 55.9)
Connections:
- --------1 pad 1: +5V -> 5v
- J2 pad 1: (no net) -> Net-(J2-PadSCL)
- J2 pad 2: (no net) -> Net-(J2-PadSDA)
- J2 pad 3: (no net) -> 5v
- J2 pad 4: (no net) -> GND
- J3 pad 1: (no net) -> Net-(J2-PadSCL)
- J3 pad 2: (no net) -> Net-(J2-PadSDA)
- J3 pad 3: (no net) -> 5v
- J3 pad 4: (no net) -> GND
- R1 pad 1: +5V -> 5v
- R1 pad 2: Net-(R1-Pad2) -> Net-(U3-Pad9)
- RV1 pad 1: +5V -> 5v
- U1 pad 3: /5v -> 5v
- U2 pad 2: +5V -> 5v
- U2 pad 3: +5V -> 5v
- U3 pad 15: Net-(R1-Pad2) -> unconnected-(U3-Pad15)
- U3 pad 7: +5V -> 5v
- U3 pad 9: unconnected-(U3-Pad9) -> Net-(U3-Pad9)
Routing:
- net +5V: track 93.7 -> 0.00 mm
- net 5v: track 0.00 -> 86.9 mm
- net GND: track 245.5 -> 221.1 mm
- net Net-(U3-Pad9): track 0.00 -> 22.4 mm
- net Net-(SW4-Pad2): track 40.0 -> 19.8 mm
- net Net-(SW3-Pad2): track 35.5 -> 18.1 mm
- net /5v: track 13.8 -> 0.00 mm
- net Net-(SW2-Pad2): track 25.7 -> 12.6 mm
- net Net-(J2-PadSDA): track 0.00 -> 10.8 mm
- net Net-(J2-PadSCL): track 0.00 -> 10.2 mm
- net Net-(R1-Pad2): track 5.08 -> 0.00 mm
- net Net-(SW1-Pad2): track 26.8 -> 23.0 mm
- net Net-(J1-Pad2): track 13.8 -> 12.7 mm
