File: Proyecto Final/Circuitos del kicad/Proyecto V1/Proyecto V1.kicad_pcb (KiCad board)
At the start: 2 copper layers, 14 parts, among them J1 12v, J2 I2C + LCD, J3 DS1307, SW1 SW_Push, SW2 SW_Push, SW3 SW_Push, SW4 SW_Push, U1 LM7805_TO220, U2 DS18B20, U3 ATmega328P-P

Commit message: save kicad
Parts:
- moved J1 14.9 mm to (164.2, 104.1)
- moved U1 9.10 mm to (159.1, 97.3)
Routing:
- net GND: track 221.1 -> 176.2 mm
- net Net-(J1-Pad2): track 12.7 -> 6.83 mm
Changed lines of the file:
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@@
   )
   (footprint "Package_TO_SOT_THT:TO-220-3_Vertical" (layer "F.Cu")
-    (at 160.02 106.361802)
+    (at 159.129094 97.306967)
     (descr "TO-220-3, Vertical, RM 2.54mm, see https://www.vishay.com/docs/66542/to-220-1.pdf")
     (tags "TO-220-3 Vertical RM 2.54mm")
@@
       (effects (font (size 1 1) (thickness 0.15)))
     )
-    (fp_text value "DS18B20" (at 1.27 2.79) (layer "F.Fab")
+    (fp_text value "DS18B20" (at 7.58 -1.16) (layer "F.Fab")
       (effects (font (size 1 1) (thickness 0.15)))
     )
@@
   )
   (footprint "TerminalBlock:TerminalBlock_bornier-2_P5.08mm" (layer "F.Cu")
-    (at 165.1 119.061802 180)
+    (at 164.209094 104.14 180)
     (descr "simple 2-pin terminal block, pitch 5.08mm, revamped version of bornier2")
     (tags "terminal block bornier2")
@@
     )
   )
-  (segment (start 160.02 119.061802) (end 160.02 106.361802) (width 1) (layer "F.Cu") (net 1))
+  (segment (start 159.129094 104.14) (end 159.129094 97.306967) (width 1) (layer "F.Cu") (net 1))
   (segment (start 137.12 99.02) (end 137.16 99.06) (width 1) (layer "F.Cu") (net 2))
-  (segment (start 165.1 119.061802) (end 162.56 116.521802) (width 1) (layer "F.Cu") (net 2))
   (segment (start 172.76 97.836402) (end 172.76 97.68) (width 0.25) (layer "F.Cu") (net 2))
-  (segment (start 167.64 104.14) (end 172.76 99.02) (width 1) (layer "F.Cu") (net 2))
   (segment (start 165.1 70.347767) (end 165.1 71.12) (width 0.5) (layer "F.Cu") (net 2))
-  (segment (start 162.56 106.361802) (end 162.56 104.14) (width 1) (layer "F.Cu") (net 2))
   (segment (start 161.735 54.975) (end 161.735 62.675) (width 0.5) (layer "F.Cu") (net 2))
   (segment (start 137.16 101.6) (end 137.16 99.06) (width 1) (layer "F.Cu") (net 2))
   (segment (start 133.44 99.02) (end 137.12 99.02) (width 1) (layer "F.Cu") (net 2))
-  (segment (start 172.76 99.02) (end 172.76 97.68) (width 1) (layer "F.Cu") (net 2))
   (segment (start 139.7 45.72) (end 147.32 45.72) (width 1) (layer "F.Cu") (net 2))
   (segment (start 137.2 53.3) (end 137.2 48.22) (width 1) (layer "F.Cu") (net 2))
   (segment (start 147.32 45.72) (end 152.4 50.8) (width 1) (layer "F.Cu") (net 2))
   (segment (start 165.617767 64.75) (end 164.622233 64.75) (width 0.5) (layer "F.Cu") (net 2))
-  (segment (start 165.1 119.061802) (end 164.781802 119.061802) (width 0.25) (layer "F.Cu") (net 2))
   (segment (start 137.16 53.34) (end 137.2 53.3) (width 1) (layer "F.Cu") (net 2))
   (segment (start 170.18 58.88) (end 168.063884 58.88) (width 0.5) (layer "F.Cu") (net 2))
@@
   (segment (start 166.35 64.017767) (end 165.617767 64.75) (width 0.5) (layer "F.Cu") (net 2))
   (segment (start 175.26 58.88) (end 170.18 58.88) (width 0.5) (layer "F.Cu") (net 2))
-  (segment (start 162.56 104.14) (end 167.64 104.14) (width 1) (layer "F.Cu") (net 2))
   (segment (start 133.44 68.54) (end 137.12 68.54) (width 1) (layer "F.Cu") (net 2))
   (segment (start 163.85 65.522233) (end 163.85 69.097767) (width 0.5) (layer "F.Cu") (net 2))
   (segment (start 157.56 50.8) (end 161.735 54.975) (width 0.5) (layer "F.Cu") (net 2))
+  (segment (start 164.209094 104.14) (end 164.209094 99.846967) (width 1) (layer "F.Cu") (net 2))
   (segment (start 165.1 71.12) (end 169.765 71.12) (width 1) (layer "F.Cu") (net 2))
   (segment (start 161.735 62.675) (end 164.216116 65.156116) (width 0.5) (layer "F.Cu") (net 2))
@@
   (segment (start 137.16 99.06) (end 137.16 83.82) (width 1) (layer "F.Cu") (net 2))
   (segment (start 137.12 83.78) (end 137.16 83.82) (width 1) (layer "F.Cu") (net 2))
-  (segment (start 162.56 116.521802) (end 162.56 106.361802) (width 1) (layer "F.Cu") (net 2))
   (segment (start 164.622233 64.75) (end 163.85 65.522233) (width 0.5) (layer "F.Cu") (net 2))
   (segment (start 169.765 71.12) (end 170.18 70.705) (width 1) (layer "F.Cu") (net 2))
   (segment (start 163.85 69.097767) (end 165.1 70.347767) (width 0.5) (layer "F.Cu") (net 2))
-  (segment (start 162.56 104.14) (end 139.7 104.14) (width 1) (layer "F.Cu") (net 2))
+  (segment (start 164.209094 99.846967) (end 161.669094 97.306967) (width 1) (layer "F.Cu") (net 2))
   (segment (start 160.06 50.8) (end 162.435 53.175) (width 0.5) (layer "F.Cu") (net 3))
   (segment (start 162.435 53.175) (end 162.435 60.835) (width 0.5) (layer "F.Cu") (net 3))
@@
   (segment (start 152.975 59.42) (end 152.4 59.42) (width 0.5) (layer "F.Cu") (net 26))
   (segment (start 155.64 59.12) (end 153.275 59.12) (width 0.5) (layer "F.Cu") (net 26))
+  (segment (start 175.3 97.68) (end 175.3 99.02) (width 1) (layer "F.Cu") (net 28))
   (segment (start 163.135 51.375) (end 162.56 50.8) (width 0.5) (layer "F.Cu") (net 28))
-  (segment (start 175.3 97.68) (end 175.3 101.56) (width 1) (layer "F.Cu") (net 28))
+  (segment (start 175.3 99.02) (end 172.72 101.6) (width 1) (layer "F.Cu") (net 28))
+  (segment (start 165.531064 98.628936) (end 164.209094 97.306967) (width 1) (layer "F.Cu") (net 28))
   (segment (start 176.135 58.517563) (end 175.497437 57.88) (width 0.5) (layer "F.Cu") (net 28))
   (segment (start 175.497437 57.88) (end 175.26 57.88) (width 0.5) (layer "F.Cu") (net 28))
@@
   (segment (start 175.26 88.9) (end 175.26 73.069009) (width 1) (layer "F.Cu") (net 28))
   (segment (start 175.26 60.117437) (end 176.135 59.242437) (width 0.5) (layer "F.Cu") (net 28))
+  (segment (start 172.72 101.6) (end 168.502128 101.6) (width 1) (layer "F.Cu") (net 28))
   (segment (start 175.26 73.069009) (end 175.26 60.117437) (width 1) (layer "F.Cu") (net 28))
   (segment (start 175.3 88.94) (end 175.26 88.9) (width 1) (layer "F.Cu") (net 28))
   (segment (start 163.135 58.42) (end 163.135 51.375) (width 0.5) (layer "F.Cu") (net 28))
-  (segment (start 170.498198 106.361802) (end 165.1 106.361802) (width 1) (layer "F.Cu") (net 28))
   (segment (start 175.3 97.68) (end 175.3 88.94) (width 1) (layer "F.Cu") (net 28))
   (segment (start 167.407767 57.88) (end 165.617767 59.67) (width 0.5) (layer "F.Cu") (net 28))
@@
   (segment (start 175.3 97.68) (end 174.03 97.68) (width 1) (layer "F.Cu") (net 28))
   (segment (start 176.135 59.242437) (end 176.135 58.517563) (width 0.5) (layer "F.Cu") (net 28))
+  (segment (start 168.502128 101.6) (end 165.531064 98.628936) (width 1) (layer "F.Cu") (net 28))
   (segment (start 175.26 73.069009) (end 170.645991 68.455) (width 1) (layer "F.Cu") (net 28))
+  (segment (start 166.031638 99.129511) (end 165.531064 98.628936) (width 1) (layer "F.Cu") (net 28))
   (segment (start 170.645991 68.455) (end 170.18 68.455) (width 1) (layer "F.Cu") (net 28))
   (segment (start 175.26 57.88) (end 170.18 57.88) (width 0.5) (layer "F.Cu") (net 28))
-  (segment (start 175.3 101.56) (end 170.498198 106.361802) (width 1) (layer "F.Cu") (net 28))
   (segment (start 157.48 70.484282) (end 157.48 71.12) (width 0.25) (layer "B.Cu") (net 28))
 )

Commit message: save kicad
Parts:
- J2, J3: footprint Connector_PinHeader_1.00mm:PinHeader_1x04_P1.00mm_Vertical -> Connector_PinSocket_2.54mm:PinSocket_1x04_P2.54mm_Vertical
- RV1: value R_Potentiometer -> Encoder; footprint Potentiometer_THT:Potentiometer_Alps_RK09Y11_Single_Horizontal -> Connector_PinSocket_1.00mm:PinSocket_1x05_P1.00mm_Vertical
- moved RV1 2.17 mm to (162.6, 48.6), turned to -90 degrees
Connections:
- --------1 pad 1: 5v -> +5V
- J2 pad 3: 5v -> +5V
- J3 pad 3: 5v -> +5V
- R1 pad 1: 5v -> +5V
- RV1 pad 1: 5v -> +5V
- U1 pad 3: 5v -> +5V
- U2 pad 2: 5v -> +5V
- U2 pad 3: 5v -> +5V
- U3 pad 20: unconnected-(U3-Pad20) -> +5V
- U3 pad 7: 5v -> +5V
Routing:
- net +5V: track 0.00 -> 96.6 mm
- net 5v: track 86.8 -> 0.00 mm
- net GND: track 176.2 -> 174.2 mm
- net Net-(U3-Pad25): track 14.8 -> 16.3 mm
- net Net-(J2-PadSDA): track 10.8 -> 10.2 mm

Commit message: save kicad
Parts:
- added C1: 20pF, Capacitor_THT:C_Disc_D5.0mm_W2.5mm_P5.00mm, F.Cu at (152.9, 70.1)
- added C2: 20pF, Capacitor_THT:C_Disc_D5.0mm_W2.5mm_P5.00mm, F.Cu at (153.0, 84.7)
- added Y1: 16MHz, Crystal:Crystal_HC49-4H_Vertical, F.Cu at (153.0, 74.9)
- Lvl_sens1: renamed from --------1; footprint Connector_PinHeader_1.00mm:PinHeader_1x03_P1.00mm_Vertical -> Connector_PinSocket_2.54mm:PinSocket_1x03_P2.54mm_Vertical
- RV1: footprint Connector_PinSocket_1.00mm:PinSocket_1x05_P1.00mm_Vertical -> Connector_PinSocket_2.54mm:PinSocket_1x05_P2.54mm_Vertical
- U1: value LM7805_TO220 -> LM7805
- s1: footprint Connector_PinHeader_1.00mm:PinHeader_1x02_P1.00mm_Vertical -> Connector_PinSocket_2.54mm:PinSocket_1x02_P2.54mm_Vertical
- moved SW1 11.8 mm to (134.2, 53.0), turned to 0 degrees
- moved RV1 3.42 mm to (166.1, 48.6)
- moved SW2 3.05 mm to (146.7, 71.5)
- moved SW3 1.70 mm to (146.7, 85.3)
- moved s1 1.33 mm to (151.4, 57.5)
- moved SW4 0.92 mm to (146.8, 99.3)
- moved Lvl_sens1 0.66 mm to (170.7, 69.0)
Connections:
- R1 pad 2: Net-(R1-Pad2) -> Net-(U3-Pad15)
- U3 pad 10: unconnected-(U3-Pad10) -> Net-(C2-Pad1)
- U3 pad 15: unconnected-(U3-Pad15) -> Net-(U3-Pad15)
- U3 pad 9: Net-(R1-Pad2) -> Net-(C1-Pad1)
Routing:
- net GND: track 174.2 -> 233.5 mm
- net +5V: track 96.6 -> 123.3 mm
- net Net-(R1-Pad2): track 22.4 -> 0.00 mm
- net Net-(C1-Pad1): track 0.00 -> 10.1 mm
- net Net-(C2-Pad1): track 0.00 -> 9.83 mm
- net Net-(SW1-Pad2): track 23.0 -> 14.4 mm
- net Net-(U3-Pad15): track 0.00 -> 5.08 mm
- net Net-(SW3-Pad2): track 18.1 -> 20.1 mm
- net Net-(U3-Pad2): track 5.09 -> 6.42 mm
- net Net-(U3-Pad23): track 5.49 -> 6.82 mm
- net Net-(SW2-Pad2): track 12.6 -> 11.3 mm
- net Net-(RV1-Pad2): track 16.3 -> 15.6 mm
- net Net-(U3-Pad3): track 5.72 -> 6.42 mm
Other:
- board outline added: 47 x 63.6 mm
- board text added: "+"
- board text added: "-"

Commit message: cum
Parts:
- removed s1: ESP8266, Connector_PinSocket_2.54mm:PinSocket_1x02_P2.54mm_Vertical
- added A1: ESP8266, Module:Adafruit_Feather, F.Cu at (166.4, 50.9)
- added U4: LD1117, Package_TO_SOT_THT:TO-220-3_Vertical, F.Cu at (167.6, 80.0)
- moved J1 31.9 mm to (151.5, 133.4)
- moved RV1 31.9 mm to (153.4, 77.8)
- moved 20pF 31.9 mm to (140.3, 113.9)
- moved 20pF 31.9 mm to (140.2, 99.3)
- moved Lvl_sens1 31.9 mm to (158.0, 98.2)
- moved R1 31.9 mm to (162.6, 118.1)
- moved SW2 31.9 mm to (134.0, 100.7)
- moved SW3 31.9 mm to (134.0, 114.5)
- moved SW4 31.9 mm to (134.1, 128.6)
- moved U1 31.9 mm to (146.4, 126.5)
- moved U2 31.9 mm to (160.1, 126.9)
- moved Y1 31.9 mm to (140.3, 104.1)
- moved J2 31.9 mm to (157.5, 85.1)
- moved J3 31.9 mm to (162.6, 85.1)
- moved SW1 31.9 mm to (121.5, 82.2)
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- renumbered C2 to 20pF, C1 to 20pF
Routing:
- net GND: track 233.5 -> 406.2 mm
- net Net-(U3-Pad3): track 6.42 -> 60.4 mm
- net Net-(U3-Pad2): track 6.42 -> 58.4 mm
- net +3V3: track 0.00 -> 35.9 mm
- net +5V: track 123.3 -> 126.2 mm
Other:
- board size 47 x 63.6 mm -> 54.6 x 90.8 mm

Commit message: cum
Routing:
- net GND: track 406.2 -> 365.8 mm
Changed lines of the file:
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@@
   (segment (start 154.94 75.32) (end 156.015 76.395) (width 0.8) (layer "B.Cu") (net 2))
   (segment (start 148.28 77.825) (end 148.28 76.5325) (width 0.8) (layer "B.Cu") (net 2))
+  (segment (start 156.8425 49) (end 158.75 50.9075) (width 0.8) (layer "B.Cu") (net 2))
   (segment (start 160.07 127.056402) (end 160.07 126.9) (width 0.8) (layer "B.Cu") (net 2))
   (segment (start 126.29 82.55) (end 126.6 82.24) (width 0.8) (layer "B.Cu") (net 2))
@@
   (segment (start 126.29 130.86) (end 126.29 128.63) (width 0.8) (layer "B.Cu") (net 2))
   (segment (start 155.35 103.28) (end 152.41 100.34) (width 0.8) (layer "B.Cu") (net 2))
-  (segment (start 171.45 125.73) (end 171.45 52.07) (width 0.8) (layer "B.Cu") (net 2))
   (segment (start 156.21 78.74) (end 157.48 80.01) (width 0.8) (layer "B.Cu") (net 2))
+  (segment (start 121 53) (end 125 49) (width 0.8) (layer "B.Cu") (net 2))
   (segment (start 126.6 82.24) (end 133.97 82.24) (width 0.8) (layer "B.Cu") (net 2))
   (segment (start 121.52 114.52) (end 126.24 114.52) (width 0.8) (layer "B.Cu") (net 2))
@@
   (segment (start 153.65 93.94) (end 153.61 93.98) (width 0.5) (layer "B.Cu") (net 2))
   (segment (start 167.64 59.7975) (end 167.64 80.01) (width 0.8) (layer "B.Cu") (net 2))
-  (segment (start 161.3975 48.26) (end 158.75 50.9075) (width 0.8) (layer "B.Cu") (net 2))
+  (segment (start 125 49) (end 156.8425 49) (width 0.8) (layer "B.Cu") (net 2))
   (segment (start 136.06 133.28) (end 128.71 133.28) (width 0.8) (layer "B.Cu") (net 2))
   (segment (start 138.07 126.28) (end 138.07 128.63) (width 0.8) (layer "B.Cu") (net 2))
@@
   (segment (start 160.62 105.89) (end 158.01 103.28) (width 0.8) (layer "B.Cu") (net 2))
   (segment (start 121.61 128.57) (end 126.23 128.57) (width 0.8) (layer "B.Cu") (net 2))
-  (segment (start 167.64 48.26) (end 161.3975 48.26) (width 0.8) (layer "B.Cu") (net 2))
   (segment (start 149.4925 75.32) (end 154.94 75.32) (width 0.8) (layer "B.Cu") (net 2))
   (segment (start 126.29 114.47) (end 126.29 100.94) (width 0.8) (layer "B.Cu") (net 2))
+  (segment (start 121 76.64) (end 121 53) (width 0.8) (layer "B.Cu") (net 2))
   (segment (start 126.07 100.72) (end 126.29 100.94) (width 0.8) (layer "B.Cu") (net 2))
   (segment (start 154.87 92.72) (end 153.65 93.94) (width 0.8) (layer "B.Cu") (net 2))
   (segment (start 151.519094 133.36) (end 151.519094 129.066967) (width 0.8) (layer "B.Cu") (net 2))
   (segment (start 153.61 93.98) (end 149.86 93.98) (width 0.5) (layer "B.Cu") (net 2))
-  (segment (start 163.82 133.36) (end 171.45 125.73) (width 0.8) (layer "B.Cu") (net 2))
   (segment (start 134.11 128.57) (end 126.23 128.57) (width 0.8) (layer "B.Cu") (net 2))
   (segment (start 138.07 131.27) (end 136.06 133.28) (width 0.8) (layer "B.Cu") (net 2))
   (segment (start 134 100.72) (end 126.07 100.72) (width 0.8) (layer "B.Cu") (net 2))
-  (segment (start 171.45 52.07) (end 167.64 48.26) (width 0.8) (layer "B.Cu") (net 2))
   (segment (start 121.47 82.24) (end 126.6 82.24) (width 0.8) (layer "B.Cu") (net 2))
   (segment (start 160.07 126.35401) (end 160.62 125.80401) (width 0.8) (layer "B.Cu") (net 2))
@@
   (segment (start 126.23 128.57) (end 126.29 128.63) (width 0.8) (layer "B.Cu") (net 2))
   (segment (start 135.453526 93.44) (end 126.29 93.44) (width 0.8) (layer "B.Cu") (net 2))
+  (segment (start 126.6 82.24) (end 121 76.64) (width 0.8) (layer "B.Cu") (net 2))
   (segment (start 121.5 100.72) (end 126.07 100.72) (width 0.8) (layer "B.Cu") (net 2))
   (segment (start 160.62 125.80401) (end 160.62 105.89) (width 0.8) (layer "B.Cu") (net 2))
-  (segment (start 151.519094 133.36) (end 163.82 133.36) (width 0.8) (layer "B.Cu") (net 2))
   (segment (start 158.75 50.9075) (end 167.64 59.7975) (width 0.8) (layer "B.Cu") (net 2))
   (segment (start 148.979094 126.526967) (end 148.979094 124.849094) (width 0.8) (layer "B.Cu") (net 2))

Commit message: Save kicad + libreria simbolo ESP
Parts:
- removed RV1: Encoder, Connector_PinSocket_2.54mm:PinSocket_1x05_P2.54mm_Vertical
- removed U4: LD1117, Package_TO_SOT_THT:TO-220-3_Vertical
- added D1: 1N4007, Diode_THT:D_DO-41_SOD81_P10.16mm_Horizontal, F.Cu at (189.6, 120.7)
- added D2: 1N4007, Diode_THT:D_DO-41_SOD81_P10.16mm_Horizontal, F.Cu at (189.6, 115.3)
- added D3: 1N4007, Diode_THT:D_DO-41_SOD81_P10.16mm_Horizontal, F.Cu at (189.6, 109.7)
- added J4: Encoder, Connector_PinSocket_2.54mm:PinSocket_1x05_P2.54mm_Vertical, F.Cu at (162.9, 97.0)
- added K1: RAYEX-L90, Relay_THT:Relay_SPDT_RAYEX-L90, F.Cu at (196.9, 60.2)
- added K2: RAYEX-L90, Relay_THT:Relay_SPDT_RAYEX-L90, F.Cu at (197.3, 120.5)
- added K3: RAYEX-L90, Relay_THT:Relay_SPDT_RAYEX-L90, F.Cu at (197.1, 90.3)
- added Q1: PN2222A, Package_TO_SOT_THT:TO-92_Inline, F.Cu at (173.9, 108.5)
- added Q2: PN2222A, Package_TO_SOT_THT:TO-92_Inline, F.Cu at (173.9, 114.1)
- added Q3: PN2222A, Package_TO_SOT_THT:TO-92_Inline, F.Cu at (173.9, 119.7)
- added R2: 1k, Resistor_THT:R_Axial_DIN0204_L3.6mm_D1.6mm_P7.62mm_Horizontal, F.Cu at (165.5, 118.5)
- added R3: 1k, Resistor_THT:R_Axial_DIN0204_L3.6mm_D1.6mm_P7.62mm_Horizontal, F.Cu at (165.5, 115.4)
- added R4: 1k, Resistor_THT:R_Axial_DIN0204_L3.6mm_D1.6mm_P7.62mm_Horizontal, F.Cu at (165.5, 112.5)
- A1: footprint Module:Adafruit_Feather -> ESP8266 LOLiN v3:ESP8266
- moved A1 18.8 mm to (148.7, 57.3)
- moved Lvl_sens1 5.01 mm to (157.8, 103.2)
- moved R1 3.14 mm to (162.7, 121.3)
- renumbered 20pF to C1, 20pF to C2
Connections:
- J2 pad 1: Net-(J2-PadSCL) -> (no net)
- J2 pad 2: Net-(J2-PadSDA) -> (no net)
- J2 pad 3: +5V -> (no net)
- J2 pad 4: GND -> (no net)
- J3 pad 1: Net-(J2-PadSCL) -> (no net)
- J3 pad 2: Net-(J2-PadSDA) -> (no net)
- J3 pad 3: +5V -> (no net)
- J3 pad 4: GND -> (no net)
- U3 pad 17: unconnected-(U3-Pad17) -> Net-(U3-Pad17)
- U3 pad 18: unconnected-(U3-Pad18) -> Net-(U3-Pad18)
- U3 pad 19: unconnected-(U3-Pad19) -> Net-(U3-Pad19)
- U3 pad 23: Net-(Lvl_sens1-Pad2) -> Net-(J4-PadCLK)
- U3 pad 24: unconnected-(U3-Pad24) -> Net-(J4-PadDT)
- U3 pad 25: Net-(RV1-Pad2) -> unconnected-(U3-Pad25)
- U3 pad 26: unconnected-(U3-Pad26) -> Net-(Lvl_sens1-Pad2)
Routing:
- net +5V: track 126.2 -> 323.6 mm
- net Net-(Q3-Pad3): track 0.00 -> 110.4 mm
- net Net-(K3-PadA1): track 0.00 -> 81.2 mm
- net GND: track 365.8 -> 440.9 mm
- net Net-(K2-PadA1): track 0.00 -> 44.0 mm
- net +3V3: track 35.9 -> 0.00 mm
- net Net-(K1-Pad11A): track 0.00 -> 21.9 mm
- net Net-(K3-Pad11A): track 0.00 -> 18.9 mm
- net Net-(K2-Pad11A): track 0.00 -> 18.9 mm
- net Net-(J4-PadCLK): track 0.00 -> 17.8 mm
- net Net-(RV1-Pad2): track 15.6 -> 0.00 mm
- net Net-(Lvl_sens1-Pad2): track 6.82 -> 22.1 mm
- net Net-(J4-PadDT): track 0.00 -> 12.3 mm
- net Net-(Q1-Pad2): track 0.00 -> 9.54 mm
- net Net-(Q3-Pad2): track 0.00 -> 9.48 mm
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Other:
- board size 54.6 x 90.8 mm -> 107.5 x 98.6 mm

Commit message: Save kikiriki
Parts:
- added C3: 330nF, Capacitor_THT:C_Disc_D5.0mm_W2.5mm_P5.00mm, F.Cu at (142.0, 131.5)
- added C4: 100nF, Capacitor_THT:C_Disc_D5.0mm_W2.5mm_P5.00mm, F.Cu at (156.0, 131.5)
- renumbered R4 to R3, R3 to R4
Connections:
- D1 pad 1: +5V -> +12V
- D2 pad 1: +5V -> +12V
- D3 pad 1: +5V -> +12V
- J1 pad 2: Net-(J1-Pad2) -> +12V
- J2 pad 1: (no net) -> Net-(J2-Pad1)
- J2 pad 2: (no net) -> Net-(J2-Pad2)
- J2 pad 3: (no net) -> +5V
- J2 pad 4: (no net) -> GND
- J3 pad 1: (no net) -> Net-(J2-Pad1)
- J3 pad 2: (no net) -> Net-(J2-Pad2)
- J3 pad 3: (no net) -> +5V
- J3 pad 4: (no net) -> GND
- J4 pad 1: (no net) -> Net-(J4-Pad1)
- J4 pad 2: (no net) -> Net-(J4-Pad2)
- J4 pad 3: (no net) -> unconnected-(J4-Pad3)
- J4 pad 4: (no net) -> +5V
- J4 pad 5: (no net) -> GND
- K1 pad A2: +5V -> +12V
- K2 pad A2: +5V -> +12V
- K3 pad A2: +5V -> +12V
- U1 pad 1: Net-(J1-Pad2) -> +12V
- U3 pad 23: Net-(J4-PadCLK) -> Net-(J4-Pad1)
- U3 pad 24: Net-(J4-PadDT) -> Net-(J4-Pad2)
- U3 pad 27: Net-(J2-PadSDA) -> Net-(J2-Pad2)
- U3 pad 28: Net-(J2-PadSCL) -> Net-(J2-Pad1)
Routing:
- net +12V: track 0.00 -> 265.1 mm
- net +5V: track 323.6 -> 95.8 mm
- net Net-(J4-Pad1): track 0.00 -> 17.9 mm
- net Net-(J4-PadCLK): track 17.8 -> 0.00 mm
- net Net-(J4-PadDT): track 12.3 -> 0.00 mm
- net Net-(J4-Pad2): track 0.00 -> 12.3 mm
- net Net-(J2-PadSDA): track 10.2 -> 0.00 mm
- net Net-(J2-PadSCL): track 10.2 -> 0.00 mm
- net Net-(J2-Pad2): track 0.00 -> 10.2 mm
- net Net-(J2-Pad1): track 0.00 -> 10.2 mm
- net Net-(J1-Pad2): track 6.83 -> 0.00 mm
- net GND: track 440.9 -> 447.2 mm
- net Net-(R2-Pad2): track 8.03 -> 8.60 mm

Commit message: cambios pene
Parts:
- removed A1: ESP8266, ESP8266 LOLiN v3:ESP8266
- added U4: NodeMCU1.0(ESP-12E), ESP8266 LOLiN v3:ESP8266, F.Cu at (151.3, 56.2)
Routing:
- net GND: track 447.2 -> 327.1 mm
- net Net-(U3-Pad2): track 54.8 -> 104.6 mm
- net Net-(U3-Pad3): track 57.0 -> 90.3 mm
- net +5V: track 95.8 -> 117.3 mm
- net Net-(D1-Pad2): track 110.4 -> 112.1 mm
- net Net-(D2-Pad2): track 81.2 -> 82.6 mm
- net Net-(D3-Pad2): track 44.0 -> 44.6 mm
Other:
- board size 107.5 x 98.6 mm -> 108.5 x 99.1 mm
