File: Proyecto Final/Circuitos del kicad/Circuito para nivel/Circuito para nivel.kicad_sch (KiCad schematic)
At the start: 10 parts, among them J1 Conn_01x05_MountingPin, J2 Conn_01x03_MountingPin, Q1 2N3904, Q2 2N3904, Q3 2N3904, Q4 2N3904

Commit message: ño
Parts:
- removed J1: Conn_01x05_MountingPin, MountingHole:MountingHole_2.1mm, symbol Connector_Generic_MountingPin:Conn_01x05_MountingPin
- removed J2: Conn_01x03_MountingPin, MountingHole:MountingHole_2.1mm, symbol Connector_Generic_MountingPin:Conn_01x03_MountingPin
- added J1: Conn_01x05, Connector_PinHeader_1.00mm:PinHeader_1x01_P1.00mm_Vertical, symbol Connector_Generic:Conn_01x05
- added J2: Conn_01x03, Connector_PinHeader_1.00mm:PinHeader_1x01_P1.00mm_Vertical, symbol Connector_Generic:Conn_01x03
- R1, R2, R3, R4: footprint Resistor_THT:R_Axial_DIN0414_L11.9mm_D4.5mm_P20.32mm_Horizontal -> Resistor_THT:R_Axial_DIN0411_L9.9mm_D3.6mm_P15.24mm_Horizontal
Connections:
- net Datos para Arduino: now also J2.2 (Pin_2)
- net GND: now also J2.3 (Pin_3)
- net VCC: now also J1.1 (Pin_1), J2.1 (Pin_1)
- net level 100%: now also J1.2 (Pin_2)
- net level 25%: now also J1.5 (Pin_5)
- net level 50%: now also J1.4 (Pin_4)
- net level 75%: now also J1.3 (Pin_3)
Other:
- moved on the sheet: Q1, Q2, Q3, Q4, R1, R2, R3, R4

Commit message: ñe
Parts:
- J1: footprint Connector_PinHeader_1.00mm:PinHeader_1x01_P1.00mm_Vertical -> Connector_PinHeader_1.00mm:PinHeader_1x05_P1.00mm_Vertical
- J2: footprint Connector_PinHeader_1.00mm:PinHeader_1x01_P1.00mm_Vertical -> Connector_PinHeader_1.00mm:PinHeader_1x03_P1.00mm_Vertical
- R1, R2, R3, R4: footprint Resistor_THT:R_Axial_DIN0411_L9.9mm_D3.6mm_P15.24mm_Horizontal -> Resistor_THT:R_Axial_DIN0207_L6.3mm_D2.5mm_P10.16mm_Horizontal
Connections:
- net VCC: now also J1.5 (Pin_5); no longer J1.1 (Pin_1)
- net level 100%: now also J1.1 (Pin_1); no longer J1.2 (Pin_2)
- net level 25%: now also J1.4 (Pin_4); no longer J1.5 (Pin_5)
- net level 50%: now also J1.3 (Pin_3); no longer J1.4 (Pin_4)
- net level 75%: now also J1.2 (Pin_2); no longer J1.3 (Pin_3)

Commit message: cum
Parts:
- J1: footprint Connector_PinHeader_1.00mm:PinHeader_1x05_P1.00mm_Vertical -> Connector_PinHeader_2.54mm:PinHeader_1x05_P2.54mm_Vertical
- J2: footprint Connector_PinHeader_1.00mm:PinHeader_1x03_P1.00mm_Vertical -> Connector_PinHeader_2.54mm:PinHeader_1x03_P2.54mm_Vertical
Changed lines of the file:
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@@
     (property "Reference" "J1" (id 0) (at 31.496 35.636 0))
     (property "Value" "Conn_01x05" (id 1) (at 31.496 38.176 0))
-    (property "Footprint" "Connector_PinHeader_1.00mm:PinHeader_1x05_P1.00mm_Vertical" (id 2) (at 31.496 46.736 0)
+    (property "Footprint" "Connector_PinHeader_2.54mm:PinHeader_1x05_P2.54mm_Vertical" (id 2) (at 31.496 46.736 0)
       (effects (font (size 1.27 1.27)) hide)
     )
@@
       (effects (font (size 1.27 1.27)) (justify left))
     )
-    (property "Footprint" "Connector_PinHeader_1.00mm:PinHeader_1x03_P1.00mm_Vertical" (id 2) (at 197.358 42.418 0)
+    (property "Footprint" "Connector_PinHeader_2.54mm:PinHeader_1x03_P2.54mm_Vertical" (id 2) (at 197.358 42.418 0)
       (effects (font (size 1.27 1.27)) hide)
     )
@@
     )
     (path "/5f4508a9-d5ee-43de-b4de-20f14d0af07d"
-      (reference "J1") (unit 1) (value "Conn_01x05") (footprint "Connector_PinHeader_1.00mm:PinHeader_1x05_P1.00mm_Vertical")
+      (reference "J1") (unit 1) (value "Conn_01x05") (footprint "Connector_PinHeader_2.54mm:PinHeader_1x05_P2.54mm_Vertical")
     )
     (path "/d8880d7e-5a80-4057-af12-2576587a5aea"
-      (reference "J2") (unit 1) (value "Conn_01x03") (footprint "Connector_PinHeader_1.00mm:PinHeader_1x03_P1.00mm_Vertical")
+      (reference "J2") (unit 1) (value "Conn_01x03") (footprint "Connector_PinHeader_2.54mm:PinHeader_1x03_P2.54mm_Vertical")
     )
     (path "/352eac11-28a4-4d80-8636-f8e5bd6a8d19"
