File: Proyecto Final/Circuitos del kicad/Circuito para nivel/Circuito para nivel.kicad_pcb (KiCad board)
At the start: 2 copper layers, 49.5 x 35 mm, 16 parts, among them Q1 2N3904, Q2 2N3904, Q3 2N3904, Q4 2N3904

Commit message: ño
Parts:
- removed the REF** at (121.5, 87.0)
- removed the REF** at (165.0, 89.5)
- removed the REF** at (121.5, 94.0)
- removed the REF** at (121.5, 80.5)
- removed the REF** at (165.0, 82.0)
- removed the REF** at (121.5, 67.0)
- removed the REF** at (121.5, 73.5)
- removed the REF** at (165.0, 75.5)
- added J1: Conn_01x05, Connector_PinHeader_1.00mm:PinHeader_1x01_P1.00mm_Vertical, F.Cu at (163.5, 65.0)
- added J2: Conn_01x03, Connector_PinHeader_1.00mm:PinHeader_1x01_P1.00mm_Vertical, F.Cu at (119.0, 89.5)
- added REF**: Pin_D0.7mm_L6.5mm_W1.8mm_FlatFork, Connector_Pin:Pin_D0.7mm_L6.5mm_W1.8mm_FlatFork, F.Cu at (120.5, 71.5)
- added REF**: Pin_D0.7mm_L6.5mm_W1.8mm_FlatFork, Connector_Pin:Pin_D0.7mm_L6.5mm_W1.8mm_FlatFork, F.Cu at (120.5, 75.0)
- added REF**: Pin_D0.7mm_L6.5mm_W1.8mm_FlatFork, Connector_Pin:Pin_D0.7mm_L6.5mm_W1.8mm_FlatFork, F.Cu at (120.5, 83.5)
- added REF**: Pin_D0.7mm_L6.5mm_W1.8mm_FlatFork, Connector_Pin:Pin_D0.7mm_L6.5mm_W1.8mm_FlatFork, F.Cu at (120.5, 79.5)
- R1, R2, R3, R4: footprint Resistor_THT:R_Axial_DIN0414_L11.9mm_D4.5mm_P20.32mm_Horizontal -> Resistor_THT:R_Axial_DIN0411_L9.9mm_D3.6mm_P15.24mm_Horizontal
- moved R4 7.53 mm to (145.4, 87.5)
- moved Q2 6.98 mm to (131.0, 72.0), turned to -90 degrees
- moved Q3 6.68 mm to (131.0, 79.0), turned to -90 degrees
- moved R3 6.59 mm to (145.6, 82.0)
- moved Q1 6.36 mm to (131.0, 65.0), turned to -90 degrees
- moved R2 6.30 mm to (145.6, 76.2)
- moved Q4 6.18 mm to (131.0, 87.5), turned to -90 degrees
- moved R1 6.09 mm to (145.6, 70.0)
Routing:
- net VCC: track 0.00 -> 95.4 mm
- net level 100%: track 0.00 -> 32.2 mm
- net level 25%: track 0.00 -> 12.1 mm
- net Net-(Q2-Pad1): track 0.00 -> 6.69 mm
- net Datos para Arduino: track 0.00 -> 6.40 mm
- net GND: track 0.00 -> 3.08 mm
- net (no net): track 0.00 -> 2.56 mm
Other:
- board outline removed
- board text added: "1k"
- board text added: "470"
- board text added: "5k6"

Commit message: ñe
Parts:
- removed REF** (x4): Pin_D0.7mm_L6.5mm_W1.8mm_FlatFork, Connector_Pin:Pin_D0.7mm_L6.5mm_W1.8mm_FlatFork
- J1: footprint Connector_PinHeader_1.00mm:PinHeader_1x01_P1.00mm_Vertical -> Connector_PinHeader_1.00mm:PinHeader_1x05_P1.00mm_Vertical
- J2: footprint Connector_PinHeader_1.00mm:PinHeader_1x01_P1.00mm_Vertical -> Connector_PinHeader_1.00mm:PinHeader_1x03_P1.00mm_Vertical
- R1, R2, R3, R4: footprint Resistor_THT:R_Axial_DIN0411_L9.9mm_D3.6mm_P15.24mm_Horizontal -> Resistor_THT:R_Axial_DIN0207_L6.3mm_D2.5mm_P10.16mm_Horizontal
- moved J1 46.6 mm to (118.0, 75.0)
- moved J2 45.1 mm to (162.0, 76.0)
- moved Q4 1.80 mm to (130.0, 86.0)
- moved Q1 1.00 mm to (130.0, 65.0)
- moved Q2 1.00 mm to (130.0, 72.0)
- moved Q3 1.00 mm to (130.0, 79.0)
- moved R1 1.00 mm to (144.6, 70.0)
- moved R2 1.00 mm to (144.6, 76.2)
- moved R3 1.00 mm to (144.6, 82.0)
- moved R4 1.00 mm to (144.4, 87.5)
Connections:
- J1 pad 1: VCC -> level 100%
Routing:
- net VCC: track 95.4 -> 192.9 mm
- net Datos para Arduino: track 6.40 -> 53.5 mm
- net Net-(Q3-Pad1): track 0.00 -> 31.1 mm
- net Net-(Q4-Pad1): track 0.00 -> 27.2 mm
- net Net-(Q2-Pad1): track 6.69 -> 32.9 mm
- net level 100%: track 32.2 -> 17.5 mm
- net level 50%: track 0.00 -> 12.9 mm
- net level 75%: track 0.00 -> 12.6 mm
- net GND: track 3.08 -> 12.8 mm
- net level 25%: track 12.1 -> 18.5 mm
- net (no net): track 2.56 -> 0.00 mm
Other:
- board outline added: 50.1 x 30 mm
- board text added: "Así estaría bien, pero no se si se tiene que espejar para que se imprima bien la placa"

Commit message: cum
Parts:
- J1: footprint Connector_PinHeader_1.00mm:PinHeader_1x05_P1.00mm_Vertical -> Connector_PinHeader_2.54mm:PinHeader_1x05_P2.54mm_Vertical
- J2: footprint Connector_PinHeader_1.00mm:PinHeader_1x03_P1.00mm_Vertical -> Connector_PinHeader_2.54mm:PinHeader_1x03_P2.54mm_Vertical
- moved R4 2.70 mm to (144.5, 84.8)
- moved R2 2.70 mm to (144.6, 73.5)
- moved R3 2.40 mm to (144.6, 79.6)
- moved R1 1.80 mm to (144.5, 68.2)
- moved J1 1.00 mm to (118.0, 74.0)
- moved J2 1.00 mm to (162.0, 75.0)
- moved Q1 1.00 mm to (130.0, 64.0)
- moved Q2 1.00 mm to (130.0, 71.0)
- moved Q3 1.00 mm to (130.0, 78.0)
- moved Q4 1.00 mm to (130.0, 85.0)
Routing:
- net VCC: track 192.9 -> 186.1 mm
- net level 25%: track 18.5 -> 13.9 mm
- net GND: track 12.8 -> 16.1 mm
- net Datos para Arduino: track 53.5 -> 51.8 mm
- net level 75%: track 12.6 -> 13.9 mm
- net Net-(Q2-Pad1): track 32.9 -> 31.9 mm
- net Net-(Q3-Pad1): track 31.1 -> 30.2 mm
- net level 50%: track 12.9 -> 12.1 mm
- net level 100%: track 17.5 -> 18.0 mm
Other:
- board text removed: "Así estaría bien, pero no se si se tiene que espejar para que se imprima bien la placa"

Commit message: cum
Changed lines of the file:
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@@
     ) (layer "Edge.Cuts") (width 0.1) (fill none))
   (gr_text "470" (at 149.9 71.1) (layer "B.Cu")
-    (effects (font (size 1.5 1.5) (thickness 0.3)) (justify mirror))
+    (effects (font (size 1.5 1.5) (thickness 0.3)))
   )
   (gr_text "1k\n" (at 150 76.3) (layer "B.Cu")
-    (effects (font (size 1.5 1.5) (thickness 0.3)) (justify mirror))
+    (effects (font (size 1.5 1.5) (thickness 0.3)))
   )
   (gr_text "1k\n" (at 150.1 65.4) (layer "B.Cu")
-    (effects (font (size 1.5 1.5) (thickness 0.3)) (justify mirror))
+    (effects (font (size 1.5 1.5) (thickness 0.3)))
   )
   (gr_text "5k6\n" (at 149.2 82.3) (layer "B.Cu")
-    (effects (font (size 1.5 1.5) (thickness 0.3)) (justify mirror))
+    (effects (font (size 1.5 1.5) (thickness 0.3)))
   )
   (segment (start 130 66.54) (end 131.34 66.54) (width 0.8) (layer "B.Cu") (net 1))
