File: Proyecto Final/Circuitos del kicad/Circuito para nivel/nueva plaqueta/Plaqueta para nivel 2/Plaqueta para nivel 2.kicad_pcb (KiCad board)
At the start: 2 copper layers, 60 x 40 mm, 20 parts, among them J1 Conn_01x05, J2 Conn_01x03, Q1 BC557, Q2 BC557, Q3 BC557, Q4 BC557, U1 ULN2003A

Commit message: COM
Parts:
- moved R8 3.45 mm to (155.0, 118.0)
- moved R10 3.44 mm to (155.0, 107.7)
- moved R12 3.44 mm to (155.0, 97.4)
- moved R6 3.25 mm to (155.0, 120.9)
- moved Q1 1.58 mm to (149.5, 110.7)
- moved Q2 1.58 mm to (149.5, 104.2)
- moved Q3 1.58 mm to (149.5, 98.2)
- moved Q4 1.58 mm to (149.5, 91.7)
- moved R13 1.27 mm to (137.5, 121.0)
- moved R5 1.25 mm to (145.5, 112.0)
- moved R11 0.75 mm to (145.5, 93.0)
- moved R7 0.75 mm to (145.5, 105.5)
- moved R9 0.75 mm to (145.5, 99.5)
- moved R2 0.52 mm to (119.0, 93.0)
- moved R3 0.52 mm to (119.0, 90.5)
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Routing:
- net GND: track 98.6 -> 105.6 mm
- net +5V: track 204.5 -> 200.8 mm
- net Net-(Q3-Pad1): track 8.13 -> 6.27 mm
- net Net-(Q4-Pad1): track 8.17 -> 6.31 mm
- net Net-(Q1-Pad1): track 11.8 -> 13.5 mm
- net Net-(R5-Pad2): track 5.43 -> 3.87 mm
- net Net-(R3-Pad1): track 19.9 -> 21.4 mm
- net Net-(Q4-Pad2): track 4.83 -> 4.00 mm
- net Net-(Q3-Pad2): track 4.83 -> 4.00 mm
- net Net-(Q2-Pad2): track 4.83 -> 4.00 mm
- net Net-(R7-Pad2): track 6.26 -> 5.66 mm
- net Net-(Q2-Pad1): track 11.2 -> 10.7 mm
