File: Proyecto Final/Circuitos del kicad/Proyecto V2/Proyecto V2 chucp.kicad_sch (KiCad schematic)
At the start: 44 parts, among them J1 12v, J2 I2C + LCD, J3 DS1307, Q1 PN2222A, Q2 PN2222A, Q3 PN2222A, SW1 SW_Push, SW2 SW_Push, SW3 SW_Push, SW4 SW_Push, U1 LM7805, U3 ATmega328P-P, Y1 16MHz

Commit message: esquematico
Changed lines of the file:
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@@
   (symbol (lib_id "Connector_Generic:Conn_01x04") (at 71.12 92.71 0) (unit 1)
     (in_bom yes) (on_board yes)
-    (property "Reference" "ESP2866-arduino1" (id 0) (at 83.82 93.9799 0)
+    (property "Reference" "ESP2866-arduino1" (id 0) (at 93.98 91.44 0)
       (effects (font (size 1.27 1.27)) (justify left))
     )
