File: Proyecto Final/Circuitos del kicad/Proyecto V2/Proyecto V2 nico.kicad_pcb (KiCad board)
At the start: 2 copper layers, 245.7 x 174.4 mm, 44 parts, among them J1 12v, J2 I2C + LCD, J3 DS1307, Q1 PN2222A, Q2 PN2222A, Q3 PN2222A, SW1 SW_Push, SW2 SW_Push, SW3 SW_Push, SW4 SW_Push, U1 LM7805, U3 ATmega328P-P, Y1 16MHz

Commit message: esquematico
Parts:
- moved D2 5.50 mm to (76.8, 139.5)
- moved Q2 5.50 mm to (84.5, 144.5)
- moved R4 5.50 mm to (85.8, 147.9)
Routing:
- net Net-(D2-Pad2): track 3.09 -> 0.00 mm
Other:
- outline, holes or cut-outs redrawn
Changed lines of the file:
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@@
   )
   (footprint "Diode_THT:D_DO-41_SOD81_P10.16mm_Horizontal" (layer "F.Cu")
-    (at 82.285 139.5)
+    (at 76.785 139.5)
     (descr "Diode, DO-41_SOD81 series, Axial, Horizontal, pin pitch=10.16mm, , length*diameter=5.2*2.7mm^2, , http://www.diodes.com/_files/packages/DO-41%20(Plastic).pdf")
     (tags "Diode DO-41_SOD81 series Axial Horizontal pin pitch 10.16mm  length 5.2mm diameter 2.7mm")
@@
   )
   (footprint "Package_TO_SOT_THT:TO-92_Inline" (layer "F.Cu")
-    (at 90 144.5)
+    (at 84.5 144.5)
     (descr "TO-92 leads in-line, narrow, oval pads, drill 0.75mm (see NXP sot054_po.pdf)")
     (tags "to-92 sc-43 sc-43a sot54 PA33 transistor")
@@
     )
     (fp_text value "1N4007" (at 15.41 -7.92 90) (layer "F.Fab")
-      (effects (font (size 1 1) (thickness 0.15)))
-    )
-    (fp_text user "K" (at 0 -2.1) (layer "F.SilkS")
-      (effects (font (size 1 1) (thickness 0.15)))
-    )
-    (fp_text user "K" (at 0 -2.1) (layer "F.Fab")
       (effects (font (size 1 1) (thickness 0.15)))
     )
@@
     (property "Sheetname" "")
     (attr through_hole)
-    (fp_text reference "Relay-2" (at -6.7934 -10.995) (layer "F.SilkS")
+    (fp_text reference "Relay-2" (at -12.2934 -10.995) (layer "F.SilkS")
       (effects (font (size 1 1) (thickness 0.15)))
     )
@@
   )
   (footprint "Resistor_THT:R_Axial_DIN0204_L3.6mm_D1.6mm_P7.62mm_Horizontal" (layer "F.Cu")
-    (at 91.32 147.95 -90)
+    (at 85.82 147.95 -90)
     (descr "Resistor, Axial_DIN0204 series, Axial, Horizontal, pin pitch=7.62mm, 0.167W, length*diameter=3.6*1.6mm^2, http://cdn-reichelt.de/documents/datenblatt/B400/1_4W%23YAG.pdf")
     (tags "Resistor Axial_DIN0204 series Axial Horizontal pin pitch 7.62mm 0.167W length 3.6mm diameter 1.6mm")
@@
   (gr_rect (start 114.58 14.32) (end 147.24 81.93) (layer "Edge.Cuts") (width 0.2) (fill none))
   (gr_rect (start 77.125 23.33) (end 32.775 93.14) (layer "Edge.Cuts") (width 0.2) (fill none))
-  (gr_rect (start 54.14 104.91) (end 140.85 188.74) (layer "Edge.Cuts") (width 0.2) (fill none))
+  (gr_rect (start 58.64 104.91) (end 140.85 188.74) (layer "Edge.Cuts") (width 0.2) (fill none))
+  (dimension (type aligned) (layer "F.Cu")
+    (pts (xy 153.28 15.152161) (xy 153.28 55.5))
+    (height 1.78)
+    (gr_text "40.3478 mm" (at 149.7 35.32608 90) (layer "F.Cu")
+      (effects (font (size 1.5 1.5) (thickness 0.3)))
+    )
+    (format (units 3) (units_format 1) (precision 4))
+    (style (thickness 0.2) (arrow_length 1.27) (text_position_mode 0) (extension_height 0.58642) (extension_offset 0.5) keep_text_aligned)
+  )
+  (dimension (type aligned) (layer "F.Cu")
+    (pts (xy 140.85 188.74) (xy 54.14 188.74))
+    (height -4.76)
+    (gr_text "86.7100 mm" (at 97.495 191.7) (layer "F.Cu")
+      (effects (font (size 1.5 1.5) (thickness 0.3)))
+    )
+    (format (units 3) (units_format 1) (precision 4))
+    (style (thickness 0.2) (arrow_length 1.27) (text_position_mode 0) (extension_height 0.58642) (extension_offset 0.5) keep_text_aligned)
+  )
+  (dimension (type aligned) (layer "F.Cu")
+    (pts (xy 140.85 188.74) (xy 140.5 105.5))
+    (height 12.499889)
+    (gr_text "83.2407 mm" (at 154.974763 147.059874 -89.75908932) (layer "F.Cu")
+      (effects (font (size 1.5 1.5) (thickness 0.3)))
+    )
+    (format (units 3) (units_format 1) (precision 4))
+    (style (thickness 0.2) (arrow_length 1.27) (text_position_mode 0) (extension_height 0.58642) (extension_offset 0.5) keep_text_aligned)
+  )
+  (dimension (type aligned) (layer "F.Cu")
+    (pts (xy 278.518479 55.5) (xy 153.28 56.30358))
+    (height -11.236098)
+    (gr_text "125.2411 mm" (at 215.959785 65.337694 0.3676275167) (layer "F.Cu")
+      (effects (font (size 1.5 1.5) (thickness 0.3)))
+    )
+    (format (units 3) (units_format 1) (precision 4))
+    (style (thickness 0.2) (arrow_length 1.27) (text_position_mode 0) (extension_height 0.58642) (extension_offset 0.5) keep_text_aligned)
+  )
+  (dimension (type aligned) (layer "F.Cu")
+    (pts (xy 114.58 14.32) (xy 114.58 81.93))
+    (height 5.08)
+    (gr_text "67.6100 mm" (at 107.7 48.125 90) (layer "F.Cu")
+      (effects (font (size 1.5 1.5) (thickness 0.3)))
+    )
+    (format (units 3) (units_format 1) (precision 4))
+    (style (thickness 0.2) (arrow_length 1.27) (text_position_mode 0) (extension_height 0.58642) (extension_offset 0.5) keep_text_aligned)
+  )
+  (dimension (type aligned) (layer "F.Cu")
+    (pts (xy 114.58 81.93) (xy 147.24 81.93))
+    (height 7.57)
+    (gr_text "32.6600 mm" (at 130.91 87.7) (layer "F.Cu")
+      (effects (font (size 1.5 1.5) (thickness 0.3)))
+    )
+    (format (units 3) (units_format 1) (precision 4))
+    (style (thickness 0.2) (arrow_length 1.27) (text_position_mode 0) (extension_height 0.58642) (extension_offset 0.5) keep_text_aligned)
+  )
   (dimension (type aligned) (layer "B.Cu")
     (pts (xy 77.225 23.36) (xy 77.225 93.16))
@@
   (segment (start 62.3 74.22) (end 64.24 72.28) (width 0.8) (layer "B.Cu") (net 12))
   (segment (start 87.755 166.98) (end 87.105 166.33) (width 0.8) (layer "B.Cu") (net 14))
-  (segment (start 92.54 144.5) (end 92.54 143.4) (width 0.8) (layer "B.Cu") (net 15))
-  (segment (start 92.445 141.49) (end 92.445 139.5) (width 0.8) (layer "B.Cu") (net 15))
   (segment (start 36.18 51.085) (end 40.47 51.085) (width 0.8) (layer "B.Cu") (net 16))
   (segment (start 35.625 47.06) (end 35.625 50.53) (width 0.8) (layer "B.Cu") (net 16))
