File: Proyecto Final/Circuitos del kicad/Proyecto V2/Proyecto V2 backup ESP.kicad_pcb (KiCad board)
At the start: 2 copper layers, 265 x 182.9 mm, 44 parts, among them J1 12v, Q1 PN2222A, Q2 PN2222A, Q3 PN2222A, SW1 SW_Push, SW2 SW_Push, SW3 SW_Push, SW4 SW_Push, U1 LM7805, U2 ESP-12E, U3 ATmega328P-P, U4 LD1117S33TR_SOT223, Y1 16MHz

Commit message: a
Parts:
- removed C5: 100nF, Capacitor_THT:C_Disc_D5.0mm_W2.5mm_P5.00mm
- removed C6: 10uF, Capacitor_THT:C_Disc_D5.0mm_W2.5mm_P5.00mm
- removed U4: LD1117S33TR_SOT223, Package_TO_SOT_THT:TO-220-3_Vertical
- added ESP2866-arduino1: Conn_02x05_Odd_Even, Connector_IDC:IDC-Header_2x05_P2.54mm_Vertical, F.Cu at (53.4, 18.6)
- added ESP8266: NodeMCU1.0(ESP-12E), ESP8266 LOLiN v3:ESP8266, F.Cu at (130.9, 45.7)
- added JESP2866-2: Conn_02x05_Odd_Even, Connector_IDC:IDC-Header_2x05_P2.54mm_Vertical, F.Cu at (125.3, 79.7)
- moved U2 144.8 mm to (143.4, 121.5), turned to 0 degrees
Connections:
- U2 pad 1: Net-(U2-Pad1) -> Net-(JESP2866-2-Pad7)
- U2 pad 15: Net-(U2-Pad15) -> Net-(JESP2866-2-Pad3)
- U2 pad 16: Net-(U2-Pad16) -> Net-(JESP2866-2-Pad5)
- U2 pad 8: Net-(C6-Pad1) -> +5V
- U3 pad 14: Net-(U2-Pad1) -> unconnected-(U3-Pad14)
- U3 pad 2: Net-(U2-Pad15) -> Net-(ESP2866-arduino1-Pad5)
- U3 pad 3: Net-(U2-Pad16) -> Net-(ESP2866-arduino1-Pad7)
Routing:
- net Net-(U2-Pad1): track 107.5 -> 0.00 mm
- net Net-(C6-Pad1): track 90.9 -> 0.00 mm
- net Net-(ESP2866-arduino1-Pad3): track 0.00 -> 47.2 mm
- net Net-(JESP2866-2-Pad7): track 0.00 -> 43.1 mm
- net +5V: track 543.6 -> 580.0 mm
- net Net-(JESP2866-2-Pad5): track 0.00 -> 35.2 mm
- net Net-(JESP2866-2-Pad3): track 0.00 -> 31.2 mm
- net Net-(U2-Pad16): track 29.3 -> 0.00 mm
- net Net-(U2-Pad15): track 19.0 -> 0.00 mm
- net Net-(ESP2866-arduino1-Pad7): track 0.00 -> 17.7 mm
- net Net-(ESP2866-arduino1-Pad5): track 0.00 -> 15.7 mm
- net Net-(Encoder/puls-arduino1-Pad7): track 178.5 -> 166.1 mm
Other:
- board size 265 x 182.9 mm -> 265 x 174.5 mm
