File: Proyecto Final/Circuitos del kicad/Proyecto V2/Proyecto V2.kicad_pcb (KiCad board)
At the start: 2 copper layers, 265 x 182.9 mm, 44 parts, among them J1 12v, Q1 PN2222A, Q2 PN2222A, Q3 PN2222A, SW1 SW_Push, SW2 SW_Push, SW3 SW_Push, SW4 SW_Push, U1 LM7805, U2 ESP-12E, U3 ATmega328P-P, U4 LD1117S33TR_SOT223, Y1 16MHz

Commit message: Cambios ESP y pines
Connections:
- Encoder/puls-arduino1 pad 1: +5V -> GND
- Encoder/puls-arduino1 pad 11: GND -> +5V
- Encoder/puls-arduino1 pad 12: GND -> +5V
- Encoder/puls-arduino1 pad 2: +5V -> GND
- Encoder/puls-arduino1 pad 3: unconnected-(Encoder/puls-arduino1-Pad3) -> Net-(U3-Pad5)
- Encoder/puls2 pad 1: +5V -> GND
- Encoder/puls2 pad 11: GND -> +5V
- Encoder/puls2 pad 12: GND -> +5V
- Encoder/puls2 pad 2: +5V -> GND
- J1 pad 1: Net-(J1-Pad1) -> GND
- U3 pad 5: unconnected-(U3-Pad5) -> Net-(U3-Pad5)
Routing:
- net +5V: track 543.6 -> 438.2 mm
- net Net-(Encoder/puls-arduino1-Pad7): track 178.5 -> 138.2 mm, vias 0 -> 2
- net Net-(U3-Pad5): track 0.00 -> 36.9 mm
- net unconnected-(U3-Pad5): track 36.5 -> 0.00 mm
- net Net-(R1-Pad1): track 29.2 -> 32.7 mm
- net Net-(C6-Pad1): track 90.9 -> 93.1 mm
- net Net-(U2-Pad1): track 107.5 -> 109.3 mm
- net Net-(Relay+DS18B20+LVL_SENS1-Pad3): track 33.8 -> 35.1 mm
- net Net-(U3-Pad4): track 43.7 -> 44.2 mm
Other:
- board size 265 x 182.9 mm -> 265 x 179.2 mm

Commit message: Cositas ricas en kikiriki
Parts:
- added J2: Conn_01x05, Connector_PinHeader_2.54mm:PinHeader_1x05_P2.54mm_Vertical, F.Cu at (42.9, 19.5)
- added J3: Conn_01x05, Connector_PinHeader_2.54mm:PinHeader_1x05_P2.54mm_Vertical, F.Cu at (108.4, 43.1)
- added J4: Conn_01x08, Connector_PinHeader_2.54mm:PinHeader_1x08_P2.54mm_Vertical, F.Cu at (121.1, 24.6)
- added J5: Conn_01x08, Connector_PinHeader_2.54mm:PinHeader_1x08_P2.54mm_Vertical, F.Cu at (143.6, 48.0)
- moved U2 97.0 mm to (132.4, 33.6), turned to 0 degrees
- moved C6 47.9 mm to (98.2, 30.3), turned to 0 degrees
- moved U4 45.7 mm to (100.7, 33.5), turned to 180 degrees
- moved C5 37.3 mm to (98.2, 38.5), turned to 0 degrees
Connections:
- C5 pad 1: +5V -> Net-(C5-Pad1)
- U2 pad 1: Net-(U2-Pad1) -> Net-(J3-Pad4)
- U2 pad 10: unconnected-(U2-Pad10) -> Net-(U2-Pad10)
- U2 pad 11: unconnected-(U2-Pad11) -> Net-(U2-Pad11)
- U2 pad 12: unconnected-(U2-Pad12) -> Net-(U2-Pad12)
- U2 pad 13: unconnected-(U2-Pad13) -> Net-(U2-Pad13)
- U2 pad 14: unconnected-(U2-Pad14) -> Net-(U2-Pad14)
- U2 pad 16: Net-(U2-Pad16) -> Net-(J5-Pad1)
- U2 pad 2: unconnected-(U2-Pad2) -> Net-(U2-Pad2)
- U2 pad 3: unconnected-(U2-Pad3) -> Net-(U2-Pad3)
- U2 pad 4: unconnected-(U2-Pad4) -> Net-(U2-Pad4)
- U2 pad 5: unconnected-(U2-Pad5) -> Net-(U2-Pad5)
- U2 pad 6: unconnected-(U2-Pad6) -> Net-(U2-Pad6)
- U2 pad 7: unconnected-(U2-Pad7) -> Net-(U2-Pad7)
- U2 pad 9: GND -> Net-(U2-Pad9)
- U3 pad 14: Net-(U2-Pad1) -> Net-(U3-Pad14)
- U3 pad 2: Net-(U2-Pad15) -> Net-(U3-Pad2)
- U3 pad 3: Net-(U2-Pad16) -> Net-(U3-Pad3)
- U4 pad 3: +5V -> Net-(C5-Pad1)
Routing:
- net Net-(U2-Pad1): track 109.3 -> 0.00 mm
- net Net-(C6-Pad1): track 93.1 -> 23.0 mm, vias 0 -> 1
- net Net-(U3-Pad14): track 0.00 -> 45.3 mm
- net Net-(J5-Pad1): track 0.00 -> 44.6 mm, vias 0 -> 1
- net Net-(U2-Pad16): track 29.3 -> 0.00 mm
- net Net-(U3-Pad3): track 0.00 -> 17.6 mm
- net Net-(U2-Pad15): track 19.0 -> 35.6 mm, vias 0 -> 1
- net Net-(U3-Pad2): track 0.00 -> 15.0 mm
- net Net-(C5-Pad1): track 0.00 -> 10.7 mm
- net Net-(Encoder/puls-arduino1-Pad7): track 138.2 -> 128.6 mm
- net Net-(U2-Pad9): track 0.00 -> 6.61 mm
- net Net-(U2-Pad14): track 0.00 -> 6.39 mm
- net Net-(U2-Pad10): track 0.00 -> 6.38 mm
- net Net-(U2-Pad13): track 0.00 -> 6.16 mm
- net Net-(U2-Pad11): track 0.00 -> 6.16 mm
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Other:
- board size 265 x 179.2 mm -> 265 x 172.9 mm

Commit message: Cambios varios
Parts:
- removed J2, J3: Conn_01x05, Connector_PinHeader_2.54mm:PinHeader_1x05_P2.54mm_Vertical
- added J6: Conn_01x06, Connector_PinHeader_2.54mm:PinHeader_1x06_P2.54mm_Vertical, F.Cu at (121.8, 21.1)
- moved C6 50.1 mm to (48.2, 27.7), turned to 90 degrees
- moved U4 48.9 mm to (52.6, 25.2), turned to -90 degrees
- moved C5 41.4 mm to (57.7, 30.2), turned to 90 degrees
- moved J4 22.1 mm to (99.2, 21.2)
- moved J5 22.1 mm to (121.7, 44.7)
- moved U2 22.1 mm to (110.5, 30.2)
- moved Encoder/puls2 10.9 mm to (223.8, 36.7)
- moved Encoder1 6.43 mm to (212.9, 13.4)
- moved U1 5.79 mm to (56.1, 77.7)
- moved C2 5.15 mm to (34.8, 58.9)
- moved C3 5.15 mm to (61.1, 82.8)
- moved Encoder/puls-arduino1 5.15 mm to (21.7, 48.7)
- moved J1 5.15 mm to (51.0, 89.5)
- moved R1 5.15 mm to (72.5, 50.9)
- moved Relay+DS18B20+LVL_SENS1 5.15 mm to (67.4, 56.0)
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Connections:
- C5 pad 1: Net-(C5-Pad1) -> +5V
- J4 pad 1: Net-(J3-Pad4) -> Net-(U3-Pad14)
- J5 pad 1: Net-(J3-Pad3) -> Net-(J5-Pad1)
- J5 pad 2: Net-(J3-Pad2) -> Net-(J5-Pad2)
- J5 pad 8: Net-(J5-Pad8) -> GND
- U2 pad 1: Net-(J3-Pad4) -> Net-(U3-Pad14)
- U2 pad 15: Net-(J3-Pad2) -> Net-(J5-Pad2)
- U2 pad 16: Net-(J3-Pad3) -> Net-(J5-Pad1)
- U2 pad 17: unconnected-(U2-Pad17) -> Net-(U2-Pad17)
- U2 pad 18: unconnected-(U2-Pad18) -> Net-(U2-Pad18)
- U2 pad 19: unconnected-(U2-Pad19) -> Net-(U2-Pad19)
- U2 pad 20: unconnected-(U2-Pad20) -> Net-(U2-Pad20)
- U2 pad 21: unconnected-(U2-Pad21) -> Net-(U2-Pad21)
- U2 pad 22: unconnected-(U2-Pad22) -> Net-(U2-Pad22)
- U2 pad 9: Net-(J5-Pad8) -> GND
- U3 pad 14: Net-(J2-Pad4) -> Net-(U3-Pad14)
- U3 pad 2: Net-(J2-Pad2) -> Net-(J5-Pad2)
- U3 pad 3: Net-(J2-Pad3) -> Net-(J5-Pad1)
- U4 pad 3: Net-(C5-Pad1) -> +5V
Routing:
- net GND: track 0.10 -> 251.6 mm, vias 0 -> 7
- net Net-(U3-Pad14): track 0.00 -> 97.4 mm, vias 0 -> 1
- net +5V: track 435.2 -> 507.4 mm
- net Net-(J2-Pad4): track 45.3 -> 0.00 mm
- net Net-(J3-Pad3): track 44.6 -> 0.00 mm, vias 1 -> 0
- net Net-(J3-Pad2): track 35.6 -> 0.00 mm, vias 1 -> 0
- net Net-(J5-Pad1): track 0.00 -> 22.6 mm, vias 0 -> 1
- net Net-(J5-Pad2): track 0.00 -> 21.3 mm, vias 0 -> 1
- net Net-(C6-Pad1): track 23.0 -> 40.6 mm
- net Net-(J2-Pad3): track 17.6 -> 0.00 mm
- net Net-(J2-Pad2): track 15.0 -> 0.00 mm
- net Net-(Encoder/puls-arduino1-Pad7): track 128.6 -> 142.6 mm
- net Net-(Encoder/puls2-Pad4): track 171.3 -> 157.8 mm
- net Net-(Encoder/puls2-Pad9): track 59.4 -> 48.4 mm
- net Net-(Encoder/puls2-Pad3): track 58.4 -> 47.5 mm
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Other:
- board size 265 x 172.9 mm -> 265.3 x 177 mm

Commit message: Agregado lib conversor y agregado a placa main
Parts:
- removed LVL_SENS1, SENS_TEMP1: Conn_01x03, TerminalBlock:TerminalBlock_bornier-3_P5.08mm
- added Salidas_sensores1: Conn_01x04, TerminalBlock:TerminalBlock_bornier-4_P5.08mm, F.Cu at (106.9, 133.3)
- added U5: BOB-12009, Conversor_logico_nivel:CONV_BOB-12009, F.Cu at (30.0, 22.4)
- moved Salida-3 6.45 mm to (106.9, 160.6)
- moved Q3 6.45 mm to (49.9, 146.0)
- moved Relay-1 6.45 mm to (74.1, 181.0)
- moved Relay-3 6.45 mm to (74.1, 124.6)
- moved Salida-2 6.45 mm to (106.9, 171.4)
- moved Q1 6.45 mm to (49.9, 134.4)
- moved Q2 6.45 mm to (49.9, 140.3)
- moved R2 6.45 mm to (44.5, 144.9)
- moved R3 6.45 mm to (45.0, 135.7)
- moved R4 6.45 mm to (44.9, 140.4)
- moved Relay1 6.45 mm to (28.7, 136.6)
- moved D1 6.45 mm to (65.7, 148.6)
- moved D2 6.45 mm to (65.7, 141.8)
- moved D3 6.45 mm to (65.7, 135.0)
- moved Relay-2 6.45 mm to (74.1, 152.8)
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Connections:
- J4 pad 8: Net-(C6-Pad1) -> Net-(J4-Pad8)
- J5 pad 1: Net-(J5-Pad1) -> Net-(U3-Pad2)
- U2 pad 16: Net-(J5-Pad1) -> Net-(U3-Pad2)
- U2 pad 8: Net-(C6-Pad1) -> Net-(J4-Pad8)
- U3 pad 2: Net-(J5-Pad2) -> Net-(U3-Pad2)
- U3 pad 3: Net-(J5-Pad1) -> Net-(U3-Pad3)
Routing:
- net +5V: track 507.4 -> 556.9 mm
- net Net-(U3-Pad3): track 0.00 -> 35.8 mm, vias 0 -> 2
- net Net-(J5-Pad1): track 22.6 -> 0.00 mm, vias 1 -> 0
- net Net-(U3-Pad2): track 0.00 -> 21.4 mm, vias 0 -> 1
- net Net-(Relay1-Pad7): track 124.1 -> 139.4 mm
- net Net-(C6-Pad1): track 40.6 -> 47.5 mm
- net Net-(Encoder/puls-arduino1-Pad7): track 142.6 -> 147.8 mm
- net Net-(J4-Pad8): track 0.00 -> 3.76 mm
- net Net-(Relay1-Pad5): track 133.3 -> 135.6 mm
- net GND: track 251.6 -> 249.5 mm
- net Net-(J4-Pad1): track 97.4 -> 99.4 mm
- net Net-(J5-Pad2): track 21.3 -> 20.2 mm, vias 1 -> 3
- net Net-(J6-Pad6): vias 1 -> 0
- net unconnected-(U5-PadLV4): vias 0 -> 1
Other:
- board size 265.3 x 177 mm -> 266.2 x 179.3 mm
