File: Proyecto Final/Circuitos del kicad/Proyecto V2/_autosave-Proyecto V2-backups/Proyecto V2.kicad_pcb (KiCad board)
At the start: 2 copper layers, 259.7 x 176.3 mm, 44 parts, among them J1 12v, J2 I2C + LCD, J3 DS1307, Q1 PN2222A, Q2 PN2222A, Q3 PN2222A, SW1 SW_Push, SW2 SW_Push, SW3 SW_Push, SW4 SW_Push, U1 LM7805, U3 ATmega328P-P, Y1 16MHz

Commit message: Cambios generales
Parts:
- moved Encoder/puls-arduino1 42.0 mm to (70.3, 44.4)
- moved C2 0.68 mm to (35.6, 64.7)
Connections:
- Encoder1 pad 1: Net-(Encoder/puls1-Pad8) -> Net-(Encoder/puls1-Pad4)
- Encoder1 pad 3: Net-(Encoder/puls1-Pad4) -> Net-(Encoder/puls1-Pad8)
Routing:
- net Net-(Encoder/puls-arduino1-Pad9): track 30.5 -> 133.5 mm
- net Net-(Encoder/puls-arduino1-Pad7): track 32.4 -> 125.0 mm
- net Net-(Encoder/puls-arduino1-Pad8): track 103.7 -> 17.3 mm
- net Net-(Encoder/puls-arduino1-Pad5): track 34.2 -> 115.8 mm
- net Net-(Encoder/puls-arduino1-Pad6): track 57.7 -> 0.00 mm
- net Net-(Encoder/puls-arduino1-Pad3): track 20.9 -> 77.4 mm
- net Net-(Encoder/puls-arduino1-Pad4): track 47.0 -> 0.00 mm
- net +5V: track 383.0 -> 401.5 mm
- net GND: track 0.27 -> 1.15 mm
Other:
- board size 259.7 x 176.3 mm -> 249.8 x 176.3 mm
