File: Proyecto Final/Circuitos del kicad/Proyecto V2/_autosave-Proyecto V2-backups/Proyecto V2.kicad_sch (KiCad schematic)
At the start: 44 parts, among them J1 12v, J2 I2C + LCD, J3 DS1307, Q1 PN2222A, Q2 PN2222A, Q3 PN2222A, SW1 SW_Push, SW2 SW_Push, SW3 SW_Push, SW4 SW_Push, U1 LM7805, U3 ATmega328P-P, Y1 16MHz

Commit message: Cambios generales
Connections:
- net at Encoder/puls1.4 (Pin_4): now also Encoder1.1 (Pin_1); no longer Encoder1.3 (Pin_3)
- net at Encoder/puls1.8 (Pin_8): now also Encoder1.3 (Pin_3); no longer Encoder1.1 (Pin_1)
Changed lines of the file:
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@@
-    (stroke (width 0) (type default) (color 0 0 0 0))
-  )
-  (wire (pts (xy 87.63 175.26) (xy 90.17 175.26))
     (stroke (width 0) (type default) (color 0 0 0 0))
   )
@@
     (stroke (width 0) (type default) (color 0 0 0 0))
   )
+  (wire (pts (xy 83.82 177.8) (xy 90.17 177.8))
+    (stroke (width 0) (type default) (color 0 0 0 0))
+  )
   (wire (pts (xy 59.69 82.55) (xy 72.644 82.55))
     (stroke (width 0) (type default) (color 0 0 0 0))
@@
     (stroke (width 0) (type default) (color 0 0 0 0))
   )
-  (wire (pts (xy 86.36 175.26) (xy 86.36 181.61))
-    (stroke (width 0) (type default) (color 0 0 0 0))
-  )
-  (wire (pts (xy 83.82 180.34) (xy 87.63 180.34))
-    (stroke (width 0) (type default) (color 0 0 0 0))
-  )
   (wire (pts (xy 177.8 147.32) (xy 177.8 143.51))
     (stroke (width 0) (type default) (color 0 0 0 0))
@@
     (stroke (width 0) (type default) (color 0 0 0 0))
   )
-  (wire (pts (xy 87.63 180.34) (xy 87.63 175.26))
-    (stroke (width 0) (type default) (color 0 0 0 0))
-  )
   (wire (pts (xy 248.92 135.89) (xy 248.92 148.59))
     (stroke (width 0) (type default) (color 0 0 0 0))
@@
     (stroke (width 0) (type default) (color 0 0 0 0))
   )
-  (wire (pts (xy 90.17 181.61) (xy 90.17 180.34))
-    (stroke (width 0) (type default) (color 0 0 0 0))
-  )
   (wire (pts (xy 170.1038 100.33) (xy 154.6098 100.33))
     (stroke (width 0) (type default) (color 0 0 0 0))
@@
     (stroke (width 0) (type default) (color 0 0 0 0))
   )
+  (wire (pts (xy 83.82 175.26) (xy 90.17 175.26))
+    (stroke (width 0) (type default) (color 0 0 0 0))
+  )
   (wire (pts (xy 85.09 110.49) (xy 85.09 151.13))
     (stroke (width 0) (type default) (color 0 0 0 0))
@@
     (stroke (width 0) (type default) (color 0 0 0 0))
   )
+  (wire (pts (xy 83.82 180.34) (xy 90.17 180.34))
+    (stroke (width 0) (type default) (color 0 0 0 0))
+  )
   (wire (pts (xy 134.62 162.56) (xy 85.09 162.56))
     (stroke (width 0) (type default) (color 0 0 0 0))
@@
     (stroke (width 0) (type default) (color 0 0 0 0))
   )
-  (wire (pts (xy 83.82 175.26) (xy 86.36 175.26))
-    (stroke (width 0) (type default) (color 0 0 0 0))
-  )
-  (wire (pts (xy 83.82 177.8) (xy 90.17 177.8))
-    (stroke (width 0) (type default) (color 0 0 0 0))
-  )
   (wire (pts (xy 134.62 148.59) (xy 134.62 110.49))
-    (stroke (width 0) (type default) (color 0 0 0 0))
-  )
-  (wire (pts (xy 86.36 181.61) (xy 90.17 181.61))
     (stroke (width 0) (type default) (color 0 0 0 0))
   )
@@
     (pin "9")
   )
-  (symbol (lib_id "Connector_Generic:Conn_02x06_Odd_Even") (at 72.39 127 0) (unit 1)
+  (symbol (lib_name "Conn_02x06_Odd_Even_1") (lib_id "Connector_Generic:Conn_02x06_Odd_Even") (at 72.39 127 0) (unit 1)
     (in_bom yes) (on_board yes)
     (property "Reference" "Encoder/puls-arduino1" (id 0) (at 73.66 138.43 0))
