File: Proyecto Final/Circuitos del kicad/Placas/Placa ESP y main/Placa_main_ESP.kicad_pcb (KiCad board)
At the start: 2 copper layers, 105.9 x 87.6 mm, 20 parts, among them J1 12v, J2 Conn_02x05_Odd_Even, J3 Conn_02x06_Odd_Even, J4 Conn_01x08, J5 Conn_01x08, J6 Conn_01x06, U1 LM7805, U2 ESP-12E, U3 ATmega328P-P, U4 LM1117-3.3, U5 BOB-12009, Y1 16MHz

Commit message: AAAAAAAAAAAAAAAAAAAAAAAAAAAAAAAAAAAAAAA
Parts:
- moved J4 15.7 mm to (188.6, 43.4)
- moved J5 15.7 mm to (211.1, 66.9)
- moved U2 15.7 mm to (199.9, 52.4)
- moved J6 15.7 mm to (211.2, 43.3)
Routing:
- net (no net): vias 0 -> 4
Other:
- board size 105.9 x 87.6 mm -> 118.7 x 100 mm
