File: Proyecto Final/Circuitos del kicad/Placas/Main y ESP test/Placa_main_ESPtest.kicad_pcb (KiCad board)
At the start: 2 copper layers, 118.7 x 100 mm, 21 parts, among them J1 12v, J2 Conn_02x05_Odd_Even, J3 Conn_02x06_Odd_Even, J4 Conn_01x08, J5 Conn_01x08, J6 Conn_01x06, U1 LM7805, U2 ESP-12E, U3 ATmega328P-P, U4 LM1117-3.3, U5 BOB-12009, Y1 16MHz

Commit message: cum
Connections:
- J2 pad 8: Net-(U3-Pad21) -> Net-(J2-Pad8)
- U3 pad 19: Net-(U3-Pad21) -> Net-(J2-Pad8)
- U3 pad 21: Net-(U3-Pad21) -> Net-(C7-Pad2)
Routing:
- net Net-(U3-Pad21): track 34.1 -> 0.00 mm
- net Net-(J2-Pad8): track 0.00 -> 30.2 mm
- net +12V: track 47.6 -> 56.1 mm
- net Net-(J2-Pad4): track 47.6 -> 44.2 mm
- net Net-(J2-Pad6): track 40.7 -> 37.4 mm
- net Net-(J3-Pad7): track 165.6 -> 163.1 mm

Commit message: cambio placa main
Parts:
- U2: footprint ESP8266-12E_ESP-12E:XCVR_ESP8266-12E_ESP-12E -> RF_Module:ESP-12E
- moved J6 151.8 mm to (61.9, 70.8), turned to 180 degrees
- moved J5 128.1 mm to (83.3, 75.8)
- moved U2 122.4 mm to (78.2, 64.7), turned to -90 degrees
- moved J4 105.8 mm to (83.3, 53.2), turned to -90 degrees
- moved U5 1.59 mm to (116.2, 65.2)
Connections:
- J4 pad 1: Net-(J4-Pad1) -> unconnected-(J4-Pad1)
- J4 pad 2: Net-(J4-Pad2) -> unconnected-(J4-Pad2)
- J4 pad 3: Net-(J4-Pad3) -> unconnected-(J4-Pad3)
- J4 pad 4: Net-(J4-Pad4) -> unconnected-(J4-Pad4)
- J4 pad 5: Net-(J4-Pad5) -> unconnected-(J4-Pad5)
- J4 pad 6: Net-(J4-Pad6) -> unconnected-(J4-Pad6)
- J4 pad 7: Net-(J4-Pad7) -> unconnected-(J4-Pad7)
- J5 pad 2: Net-(J5-Pad2) -> Net-(U5-PadLV1)
- J5 pad 3: Net-(J5-Pad3) -> unconnected-(J5-Pad3)
- J5 pad 4: Net-(J5-Pad4) -> unconnected-(J5-Pad4)
- J5 pad 5: Net-(J5-Pad5) -> unconnected-(J5-Pad5)
- J5 pad 6: Net-(J5-Pad6) -> unconnected-(J5-Pad6)
- J5 pad 7: Net-(J5-Pad7) -> unconnected-(J5-Pad7)
- J6 pad 1: Net-(J6-Pad1) -> unconnected-(J6-Pad1)
- J6 pad 2: Net-(J6-Pad2) -> unconnected-(J6-Pad2)
- J6 pad 3: Net-(J6-Pad3) -> unconnected-(J6-Pad3)
- J6 pad 4: Net-(J6-Pad4) -> unconnected-(J6-Pad4)
- J6 pad 5: Net-(J6-Pad5) -> unconnected-(J6-Pad5)
- J6 pad 6: Net-(J6-Pad6) -> unconnected-(J6-Pad6)
- U2 pad 1: Net-(J4-Pad1) -> unconnected-(U2-Pad1)
- U2 pad 10: Net-(J5-Pad7) -> unconnected-(U2-Pad10)
- U2 pad 11: Net-(J5-Pad6) -> unconnected-(U2-Pad11)
- U2 pad 12: Net-(J5-Pad5) -> unconnected-(U2-Pad12)
- U2 pad 13: Net-(J5-Pad4) -> unconnected-(U2-Pad13)
- U2 pad 14: Net-(J5-Pad3) -> unconnected-(U2-Pad14)
- U2 pad 15: Net-(J5-Pad2) -> GND
- U2 pad 16: Net-(J5-Pad1) -> unconnected-(U2-Pad16)
- U2 pad 17: Net-(J6-Pad6) -> unconnected-(U2-Pad17)
- U2 pad 18: Net-(J6-Pad5) -> unconnected-(U2-Pad18)
- U2 pad 19: Net-(J6-Pad4) -> unconnected-(U2-Pad19)
- U2 pad 2: Net-(J4-Pad2) -> unconnected-(U2-Pad2)
- U2 pad 20: Net-(J6-Pad3) -> unconnected-(U2-Pad20)
- U2 pad 21: Net-(J6-Pad2) -> Net-(U5-PadLV1)
- U2 pad 22: Net-(J6-Pad1) -> Net-(J5-Pad1)
- U2 pad 3: Net-(J4-Pad3) -> unconnected-(U2-Pad3)
- U2 pad 4: Net-(J4-Pad4) -> unconnected-(U2-Pad4)
- U2 pad 5: Net-(J4-Pad5) -> unconnected-(U2-Pad5)
- U2 pad 6: Net-(J4-Pad6) -> unconnected-(U2-Pad6)
- U2 pad 7: Net-(J4-Pad7) -> unconnected-(U2-Pad7)
- U2 pad 9: GND -> unconnected-(U2-Pad9)
- U3 pad 14: Net-(J4-Pad1) -> unconnected-(U3-Pad14)
- U3 pad 21: Net-(C7-Pad2) -> unconnected-(U3-Pad21)
Routing:
- net Net-(J4-Pad1): track 108.8 -> 0.00 mm, vias 1 -> 0
- net unconnected-(U3-Pad14): track 0.00 -> 104.2 mm, vias 0 -> 1
- net Net-(J5-Pad2): track 21.5 -> 13.6 mm, vias 3 -> 2
- net Net-(J5-Pad1): track 21.4 -> 14.1 mm
- net Net-(J5-Pad3): track 6.39 -> 0.00 mm
- net Net-(J5-Pad7): track 6.38 -> 0.00 mm
- net Net-(J5-Pad4): track 6.16 -> 0.00 mm
- net Net-(J5-Pad6): track 6.16 -> 0.00 mm
- net Net-(J5-Pad5): track 5.94 -> 0.00 mm
- net Net-(J6-Pad1): track 4.69 -> 0.00 mm, vias 1 -> 0
- net Net-(J4-Pad2): track 4.46 -> 0.00 mm
- net Net-(J6-Pad2): track 4.39 -> 0.00 mm
- net Net-(J4-Pad7): track 4.33 -> 0.00 mm
- net Net-(J4-Pad3): track 4.24 -> 0.00 mm
- net Net-(J6-Pad3): track 4.17 -> 0.00 mm
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Other:
- board size 118.7 x 100 mm -> 112.2 x 85.3 mm
