File: Proyecto Final/Circuitos del kicad/Placas/Main y ESP test/Placa_main_ESPtest.kicad_sch (KiCad schematic)
At the start: 22 parts, among them J1 12v, J2 Conn_02x05_Odd_Even, J3 Conn_02x06_Odd_Even, J4 Conn_01x08, J5 Conn_01x08, J6 Conn_01x06, U1 LM7805, U2 ESP-12E, U3 ATmega328P-P, U4 LM1117-3.3, U5 BOB-12009, Y1 16MHz

Commit message: cambio placa main
Parts:
- removed C7: 100nF, Capacitor_THT:C_Disc_D5.0mm_W2.5mm_P5.00mm, symbol Device:C
- removed U2: ESP-12E, ESP8266-12E_ESP-12E:XCVR_ESP8266-12E_ESP-12E, symbol ESP8266:ESP-12E
- added U2: ESP-12E, RF_Module:ESP-12E, symbol RF_Module:ESP-12E
Connections:
- net +12V: now also J2.10 (Pin_10); no longer J2.2 (Pin_2)
- net +5V: now also J2.9 (Pin_9); no longer J2.1 (Pin_1)
- net GND: now also J2.1 (Pin_1), J2.2 (Pin_2), U2.15 (GND); no longer J2.10 (Pin_10), J2.9 (Pin_9)
- net at J5.2 (Pin_2), U5.LV1: now also U2.21 (GPIO3/RXD)
- net at J5.1 (Pin_1), U3.2 (PD0): now also U2.22 (GPIO1/TXD)
- net at J4.1 (Pin_1): no longer U3.14 (PB0)
- net at J4.8 (Pin_8): now also U2.8 (VCC)
- no-connect marks 10 -> 49
Other:
- note removed: "RST"
- moved on the sheet: J6

Commit message: La pc del colegio rompio el archivo
Parts:
- removed U2: ESP-12E, RF_Module:ESP-12E, symbol RF_Module:ESP-12E
- added C7: 100nF, Capacitor_THT:C_Disc_D5.0mm_W2.5mm_P5.00mm, symbol Device:C
- added U2: ESP-12E, ESP8266-12E_ESP-12E:XCVR_ESP8266-12E_ESP-12E, symbol ESP8266:ESP-12E
Connections:
- net +12V: now also J2.2 (Pin_2); no longer J2.10 (Pin_10)
- net +5V: now also J2.1 (Pin_1); no longer J2.9 (Pin_9)
- net GND: now also J2.10 (Pin_10), J2.9 (Pin_9), C7.1, U2.9 (GND); no longer J2.1 (Pin_1), J2.2 (Pin_2)
- net at J5.2 (Pin_2), U5.LV1: now also U2.15 (RXD)
- net at J5.1 (Pin_1), U3.2 (PD0): now also U2.16 (TXD)
- net at J5.3 (Pin_3): now also U2.14 (GPIO5)
- net at J5.4 (Pin_4): now also U2.13 (GPIO4)
- net at J5.5 (Pin_5): now also U2.12 (GPIO0)
- net at J5.6 (Pin_6): now also U2.11 (GPIO2)
- net at J5.7 (Pin_7): now also U2.10 (GPIO15)
- net at J6.1 (Pin_1): now also U2.22 (SCLK)
- net at J6.2 (Pin_2): now also U2.21 (MOSI)
- net at J6.3 (Pin_3): now also U2.20 (GPIO10)
- net at J6.4 (Pin_4): now also U2.19 (GPIO9)
- net at J6.5 (Pin_5): now also U2.18 (MISO)
- net at J6.6 (Pin_6): now also U2.17 (CS0)
- net at J4.1 (Pin_1): now also U3.14 (PB0), U2.1 (REST)
- net at J4.2 (Pin_2): now also U2.2 (ADC)
- net at J4.3 (Pin_3): now also U2.3 (CH_PD)
- net at J4.4 (Pin_4): now also U2.4 (GPIO16)
- net at J4.5 (Pin_5): now also U2.5 (GPIO14)
- net at J4.6 (Pin_6): now also U2.6 (GPIO12)
- net at J4.7 (Pin_7): now also U2.7 (GPIO13)
- net at J4.8 (Pin_8): now also U2.8 (VCC)
- net at U3.21 (AREF): now also C7.2
- no-connect marks 49 -> 10
Other:
- note added: "RST"
- moved on the sheet: J6

Commit message: Placas bien subidas
Parts:
- removed C7: 100nF, Capacitor_THT:C_Disc_D5.0mm_W2.5mm_P5.00mm, symbol Device:C
- removed U2: ESP-12E, ESP8266-12E_ESP-12E:XCVR_ESP8266-12E_ESP-12E, symbol ESP8266:ESP-12E
- added U2: ESP-12E, RF_Module:ESP-12E, symbol RF_Module:ESP-12E
Connections:
- net +12V: now also J2.10 (Pin_10); no longer J2.2 (Pin_2)
- net +5V: now also J2.9 (Pin_9); no longer J2.1 (Pin_1)
- net GND: now also J2.1 (Pin_1), J2.2 (Pin_2), U2.15 (GND); no longer J2.10 (Pin_10), J2.9 (Pin_9)
- net at J5.2 (Pin_2), U5.LV1: now also U2.21 (GPIO3/RXD)
- net at J5.1 (Pin_1), U3.2 (PD0): now also U2.22 (GPIO1/TXD)
- net at J4.1 (Pin_1): no longer U3.14 (PB0)
- net at J4.8 (Pin_8): now also U2.8 (VCC)
- net at U3.26 (PC3): now also J2.7 (Pin_7); no longer J2.3 (Pin_3)
- no-connect marks 10 -> 49
Other:
- note removed: "RST"
- moved on the sheet: J6

Commit message: Cambios ancho de agujeros placa main
Parts:
- J4, J5: footprint Connector_PinHeader_2.54mm:PinHeader_1x08_P2.54mm_Vertical -> Connector_PinSocket_2.54mm:PinSocket_1x08_P2.54mm_Vertical
- J6: footprint Connector_PinHeader_2.54mm:PinHeader_1x06_P2.54mm_Vertical -> Connector_PinSocket_2.54mm:PinSocket_1x06_P2.54mm_Vertical
Changed lines of the file:
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@@
       (effects (font (size 1.27 1.27)) (justify left))
     )
-    (property "Footprint" "Connector_PinHeader_2.54mm:PinHeader_1x08_P2.54mm_Vertical" (id 2) (at 229.235 123.317 0)
+    (property "Footprint" "Connector_PinSocket_2.54mm:PinSocket_1x08_P2.54mm_Vertical" (id 2) (at 229.235 123.317 0)
       (effects (font (size 1.27 1.27)) hide)
     )
@@
     (property "Reference" "J6" (id 0) (at 197.993 160.02 90))
     (property "Value" "Conn_01x06" (id 1) (at 197.993 162.56 90))
-    (property "Footprint" "Connector_PinHeader_2.54mm:PinHeader_1x06_P2.54mm_Vertical" (id 2) (at 199.263 156.21 0)
+    (property "Footprint" "Connector_PinSocket_2.54mm:PinSocket_1x06_P2.54mm_Vertical" (id 2) (at 199.263 156.21 0)
       (effects (font (size 1.27 1.27)) hide)
     )
@@
       (effects (font (size 1.27 1.27)) hide)
     )
-    (property "Footprint" "Connector_PinHeader_2.54mm:PinHeader_1x08_P2.54mm_Vertical" (id 2) (at 169.545 125.095 0)
+    (property "Footprint" "Connector_PinSocket_2.54mm:PinSocket_1x08_P2.54mm_Vertical" (id 2) (at 169.545 125.095 0)
       (effects (font (size 1.27 1.27)) hide)
     )
@@
     )
     (path "/b221cb34-347c-4dd4-9279-103a258c41cf"
-      (reference "J4") (unit 1) (value "Conn_01x08") (footprint "Connector_PinHeader_2.54mm:PinHeader_1x08_P2.54mm_Vertical")
+      (reference "J4") (unit 1) (value "Conn_01x08") (footprint "Connector_PinSocket_2.54mm:PinSocket_1x08_P2.54mm_Vertical")
     )
     (path "/1c714670-6c43-4ef9-a98b-4206a0351ce4"
-      (reference "J5") (unit 1) (value "Conn_01x08") (footprint "Connector_PinHeader_2.54mm:PinHeader_1x08_P2.54mm_Vertical")
+      (reference "J5") (unit 1) (value "Conn_01x08") (footprint "Connector_PinSocket_2.54mm:PinSocket_1x08_P2.54mm_Vertical")
     )
     (path "/9266ad98-56ad-4979-a534-eef1d9b8c163"
-      (reference "J6") (unit 1) (value "Conn_01x06") (footprint "Connector_PinHeader_2.54mm:PinHeader_1x06_P2.54mm_Vertical")
+      (reference "J6") (unit 1) (value "Conn_01x06") (footprint "Connector_PinSocket_2.54mm:PinSocket_1x06_P2.54mm_Vertical")
     )
     (path "/6a730b26-141b-4550-bfbd-6131095893ab"
