File: Proyecto Final/Circuitos del kicad/Placas/Placa pulsadores/Placa_pulsadores.kicad_pcb (KiCad board)
At the start: 2 copper layers, 129.7 x 34.4 mm, 10 parts, among them SW1 SW_Push, SW2 SW_Push, SW3 SW_Push, SW4 SW_Push

Commit message: Cambios placa pulsadores
Parts:
- removed Encoder/puls2: Conn_02x06_Odd_Even, ENCODER+PULS:ENCODER+PULS
- added J1: Conn_02x06_Odd_Even, Connector_IDC:IDC-Header_2x06_P2.54mm_Vertical, F.Cu at (153.3, 98.1)
- R5, R6, R7, R8: footprint Resistor_THT:R_Axial_DIN0204_L3.6mm_D1.6mm_P5.08mm_Horizontal -> Resistor_THT:R_Axial_DIN0207_L6.3mm_D2.5mm_P5.08mm_Vertical
- moved R8 1.36 mm to (141.0, 93.0)
- moved R7 0.82 mm to (144.8, 93.0)
- moved R5 0.64 mm to (152.1, 93.0)
- moved R6 0.25 mm to (148.4, 93.0)
Routing:
- net Net-(J1-Pad3): track 47.5 -> 60.5 mm
- net Net-(J1-Pad5): track 34.1 -> 47.0 mm
- net Net-(J1-Pad9): track 48.4 -> 60.4 mm
- net Net-(J1-Pad7): track 35.3 -> 47.2 mm

Commit message: Amplie distancia de resistencias
Parts:
- moved R8 3.05 mm to (137.9, 93.0)
- moved R7 1.27 mm to (143.5, 93.0)
- moved R5 1.02 mm to (153.2, 93.0)
Routing:
- net Net-(J1-Pad3): track 60.5 -> 62.4 mm
- net Net-(J1-Pad5): track 47.0 -> 48.5 mm
- net Net-(J1-Pad9): track 60.4 -> 61.9 mm
- net Net-(J1-Pad7): track 47.2 -> 48.1 mm
Changed lines of the file:
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@@
   )
   (footprint "Resistor_THT:R_Axial_DIN0207_L6.3mm_D2.5mm_P5.08mm_Vertical" (layer "F.Cu")
-    (at 144.78 92.964 90)
+    (at 143.51 92.964 90)
     (descr "Resistor, Axial_DIN0207 series, Axial, Vertical, pin pitch=5.08mm, 0.25W = 1/4W, length*diameter=6.3*2.5mm^2, http://cdn-reichelt.de/documents/datenblatt/B400/1_4W%23YAG.pdf")
     (tags "Resistor Axial_DIN0207 series Axial Vertical pin pitch 5.08mm 0.25W = 1/4W length 6.3mm diameter 2.5mm")
@@
   )
   (footprint "Resistor_THT:R_Axial_DIN0207_L6.3mm_D2.5mm_P5.08mm_Vertical" (layer "F.Cu")
-    (at 140.97 92.964 90)
+    (at 137.922 92.964 90)
     (descr "Resistor, Axial_DIN0207 series, Axial, Vertical, pin pitch=5.08mm, 0.25W = 1/4W, length*diameter=6.3*2.5mm^2, http://cdn-reichelt.de/documents/datenblatt/B400/1_4W%23YAG.pdf")
     (tags "Resistor Axial_DIN0207 series Axial Vertical pin pitch 5.08mm 0.25W = 1/4W length 6.3mm diameter 2.5mm")
@@
   )
   (footprint "Resistor_THT:R_Axial_DIN0207_L6.3mm_D2.5mm_P5.08mm_Vertical" (layer "F.Cu")
-    (at 152.146 92.964 90)
+    (at 153.162 92.964 90)
     (descr "Resistor, Axial_DIN0207 series, Axial, Vertical, pin pitch=5.08mm, 0.25W = 1/4W, length*diameter=6.3*2.5mm^2, http://cdn-reichelt.de/documents/datenblatt/B400/1_4W%23YAG.pdf")
     (tags "Resistor Axial_DIN0207 series Axial Vertical pin pitch 5.08mm 0.25W = 1/4W length 6.3mm diameter 2.5mm")
@@
   (via (at 205.19 74.93) (size 4) (drill 3.5) (layers "F.Cu" "B.Cu") (free) (net 0))
   (via (at 205.51 104.43) (size 4) (drill 3.5) (layers "F.Cu" "B.Cu") (free) (net 0))
+  (segment (start 92.114 98.044) (end 86.35 92.28) (width 1.2) (layer "B.Cu") (net 2))
+  (segment (start 140.544 98.044) (end 92.114 98.044) (width 1.2) (layer "B.Cu") (net 2))
+  (segment (start 86.42 85.76) (end 122.49 85.76) (width 1.2) (layer "B.Cu") (net 2))
+  (segment (start 86.35 82.39) (end 88.61 80.13) (width 1.2) (layer "B.Cu") (net 2))
+  (segment (start 140.58 98.08) (end 140.544 98.044) (width 1.2) (layer "B.Cu") (net 2))
   (segment (start 88.61 80.13) (end 145.86 80.13) (width 1.2) (layer "B.Cu") (net 2))
-  (segment (start 145.86 80.13) (end 150.065 75.925) (width 1.2) (layer "B.Cu") (net 2))
-  (segment (start 138.18 95.68) (end 104.47 95.68) (width 1.2) (layer "B.Cu") (net 2))
-  (segment (start 86.35 82.39) (end 88.61 80.13) (width 1.2) (layer "B.Cu") (net 2))
-  (segment (start 150.065 75.925) (end 150.065 74.78) (width 1.2) (layer "B.Cu") (net 2))
-  (segment (start 86.42 85.76) (end 122.49 85.76) (width 1.2) (layer "B.Cu") (net 2))
   (segment (start 86.35 92.28) (end 86.35 82.39) (width 1.2) (layer "B.Cu") (net 2))
   (segment (start 140.58 98.08) (end 140.58 100.62) (width 1.2) (layer "B.Cu") (net 2))
-  (segment (start 140.58 98.08) (end 138.18 95.68) (width 1.2) (layer "B.Cu") (net 2))
-  (segment (start 104.47 95.68) (end 89.75 95.68) (width 1.2) (layer "B.Cu") (net 2))
-  (segment (start 89.75 95.68) (end 86.35 92.28) (width 1.2) (layer "B.Cu") (net 2))
+  (segment (start 150.065 75.925) (end 150.065 74.78) (width 1.2) (layer "B.Cu") (net 2))
   (segment (start 124.614 87.884) (end 152.146 87.884) (width 1.2) (layer "B.Cu") (net 2))
+  (segment (start 145.86 80.13) (end 150.065 75.925) (width 1.2) (layer "B.Cu") (net 2))
   (segment (start 122.49 85.76) (end 124.614 87.884) (width 1.2) (layer "B.Cu") (net 2))
   (segment (start 145.7 105.66) (end 150.74 100.62) (width 1) (layer "B.Cu") (net 3))
@@
   (segment (start 84.65 99.97) (end 84.65 81.55) (width 1) (layer "B.Cu") (net 5))
   (segment (start 87.13 102.45) (end 84.65 99.97) (width 1) (layer "B.Cu") (net 5))
-  (segment (start 154.432 93.98) (end 152.908 95.504) (width 1) (layer "B.Cu") (net 6))
+  (segment (start 155.448 95.504) (end 157.988 92.964) (width 1) (layer "B.Cu") (net 6))
+  (segment (start 152.4 95.504) (end 155.448 95.504) (width 1) (layer "B.Cu") (net 6))
+  (segment (start 150.74 97.164) (end 152.4 95.504) (width 1) (layer "B.Cu") (net 6))
   (segment (start 186.446 92.964) (end 191.19 88.22) (width 1) (layer "B.Cu") (net 6))
-  (segment (start 152.146 92.964) (end 186.446 92.964) (width 1) (layer "B.Cu") (net 6))
+  (segment (start 157.988 92.964) (end 186.446 92.964) (width 1) (layer "B.Cu") (net 6))
+  (segment (start 153.162 92.964) (end 157.988 92.964) (width 1) (layer "B.Cu") (net 6))
   (segment (start 203.69 88.22) (end 191.19 88.22) (width 1) (layer "B.Cu") (net 6))
   (segment (start 150.74 97.164) (end 150.74 98.08) (width 0.8) (layer "B.Cu") (net 6))
-  (segment (start 152.4 95.504) (end 150.74 97.164) (width 1) (layer "B.Cu") (net 6))
-  (segment (start 154.432 92.964) (end 154.432 93.98) (width 1) (layer "B.Cu") (net 6))
-  (segment (start 152.908 95.504) (end 152.4 95.504) (width 1) (layer "B.Cu") (net 6))
-  (segment (start 150.114 91.44) (end 150.014 91.34) (width 1) (layer "B.Cu") (net 7))
+  (segment (start 151.13 90.678) (end 150.622 90.678) (width 1) (layer "B.Cu") (net 7))
+  (segment (start 151.13 93.98) (end 151.13 90.678) (width 1) (layer "B.Cu") (net 7))
+  (segment (start 151.184 90.17) (end 150.014 91.34) (width 1) (layer "B.Cu") (net 7))
+  (segment (start 148.2 96.91) (end 151.13 93.98) (width 1) (layer "B.Cu") (net 7))
   (segment (start 150.014 91.34) (end 148.39 92.964) (width 1) (layer "B.Cu") (net 7))
-  (segment (start 150.368 90.986) (end 150.014 91.34) (width 1) (layer "B.Cu") (net 7))
-  (segment (start 170.568 90.932) (end 150.368 90.932) (width 1) (layer "B.Cu") (net 7))
+  (segment (start 148.2 98.08) (end 148.2 96.91) (width 1) (layer "B.Cu") (net 7))
   (segment (start 185.78 88.22) (end 173.28 88.22) (width 1) (layer "B.Cu") (net 7))
-  (segment (start 148.2 97.14) (end 150.114 95.226) (width 1) (layer "B.Cu") (net 7))
-  (segment (start 150.368 90.932) (end 150.368 90.986) (width 1) (layer "B.Cu") (net 7))
-  (segment (start 150.114 95.226) (end 150.114 91.44) (width 1) (layer "B.Cu") (net 7))
-  (segment (start 148.2 98.08) (end 148.2 97.14) (width 0.8) (layer "B.Cu") (net 7))
-  (segment (start 173.28 88.22) (end 170.568 90.932) (width 1) (layer "B.Cu") (net 7))
-  (segment (start 145.66 97.146) (end 143.002 94.488) (width 1) (layer "B.Cu") (net 8))
-  (segment (start 143.002 91.186) (end 123.246 91.186) (width 1) (layer "B.Cu") (net 8))
-  (segment (start 143.002 94.488) (end 143.002 91.44) (width 1) (layer "B.Cu") (net 8))
-  (segment (start 145.66 98.08) (end 145.66 97.146) (width 0.8) (layer "B.Cu") (net 8))
-  (segment (start 123.246 91.186) (end 120.2 88.14) (width 1) (layer "B.Cu") (net 8))
+  (segment (start 171.33 90.17) (end 151.184 90.17) (width 1) (layer "B.Cu") (net 7))
+  (segment (start 173.28 88.22) (end 171.33 90.17) (width 1) (layer "B.Cu") (net 7))
+  (segment (start 145.66 98.08) (end 145.66 97.146) (width 1) (layer "B.Cu") (net 8))
+  (segment (start 145.66 97.146) (end 144.526 96.012) (width 1) (layer "B.Cu") (net 8))
+  (segment (start 140.208 90.678) (end 141.224 90.678) (width 1) (layer "B.Cu") (net 8))
+  (segment (start 141.224 90.678) (end 143.51 92.964) (width 1) (layer "B.Cu") (net 8))
+  (segment (start 122.738 90.678) (end 140.208 90.678) (width 1) (layer "B.Cu") (net 8))
+  (segment (start 120.2 88.14) (end 122.738 90.678) (width 1) (layer "B.Cu") (net 8))
+  (segment (start 143.383 96.012) (end 140.208 92.837) (width 1) (layer "B.Cu") (net 8))
   (segment (start 107.7 88.14) (end 120.2 88.14) (width 1) (layer "B.Cu") (net 8))
-  (segment (start 144.78 92.964) (end 143.002 91.186) (width 1) (layer "B.Cu") (net 8))
-  (segment (start 143.002 91.44) (end 142.748 91.186) (width 0.8) (layer "B.Cu") (net 8))
-  (segment (start 138.938 93.218) (end 138.938 93.818) (width 1) (layer "B.Cu") (net 9))
+  (segment (start 144.526 96.012) (end 143.383 96.012) (width 1) (layer "B.Cu") (net 8))
+  (segment (start 140.208 92.837) (end 140.208 90.678) (width 1) (layer "B.Cu") (net 8))
+  (segment (start 106.604 92.964) (end 101.78 88.14) (width 1) (layer "B.Cu") (net 9))
+  (segment (start 136.398 95.504) (end 134.112 93.218) (width 1) (layer "B.Cu") (net 9))
+  (segment (start 134.112 92.964) (end 106.604 92.964) (width 1) (layer "B.Cu") (net 9))
+  (segment (start 143.1 97.98) (end 140.624 95.504) (width 1) (layer "B.Cu") (net 9))
+  (segment (start 137.922 92.964) (end 134.112 92.964) (width 1) (layer "B.Cu") (net 9))
   (segment (start 89.28 88.14) (end 101.78 88.14) (width 1) (layer "B.Cu") (net 9))
-  (segment (start 138.938 93.818) (end 143.1 97.98) (width 1) (layer "B.Cu") (net 9))
-  (segment (start 140.97 92.964) (end 140.744 93.19) (width 1) (layer "B.Cu") (net 9))
-  (segment (start 140.744 93.19) (end 106.83 93.19) (width 1) (layer "B.Cu") (net 9))
-  (segment (start 106.83 93.19) (end 101.78 88.14) (width 1) (layer "B.Cu") (net 9))
+  (segment (start 134.112 93.218) (end 134.112 92.964) (width 1) (layer "B.Cu") (net 9))
+  (segment (start 140.624 95.504) (end 136.398 95.504) (width 1) (layer "B.Cu") (net 9))
   (zone (net 1) (net_name "GND") (layer "B.Cu") (hatch edge 0.508)
-    (connect_pads (clearance 1))
+    (connect_pads yes (clearance 1))
     (min_thickness 0.254) (filled_areas_thickness no)
     (fill yes (thermal_gap 0.508) (thermal_bridge_width 0.508))
