File: Proyecto Final/Circuitos del kicad/Placas/Placa pulsadores/Placa_pulsadores.kicad_sch (KiCad schematic)
At the start: 10 parts, among them SW1 SW_Push, SW2 SW_Push, SW3 SW_Push, SW4 SW_Push

Commit message: Cambios placa pulsadores
Parts:
- removed Encoder/puls2: Conn_02x06_Odd_Even, ENCODER+PULS:ENCODER+PULS, symbol ENCODER+PULS:Conn_02x06_Odd_Even
- added J1: Conn_02x06_Odd_Even, Connector_IDC:IDC-Header_2x06_P2.54mm_Vertical, symbol Connector_Generic:Conn_02x06_Odd_Even
- R5, R6, R7, R8: footprint Resistor_THT:R_Axial_DIN0204_L3.6mm_D1.6mm_P5.08mm_Horizontal -> Resistor_THT:R_Axial_DIN0207_L6.3mm_D2.5mm_P5.08mm_Vertical
Connections:
- net +5V: now also J1.11 (Pin_11), J1.12 (Pin_12)
- net GND: now also J1.1 (Pin_1), J1.2 (Pin_2)
- net at R7.1, SW2.2: now also J1.7 (Pin_7)
- net at R8.1, SW1.2: now also J1.9 (Pin_9)
- net at R6.1, SW3.2: now also J1.5 (Pin_5)
- net at R5.1, SW4.2: now also J1.3 (Pin_3)
- net at Encoder1.1 (Pin_1): now also J1.4 (Pin_4)
- net at Encoder1.2 (Pin_2): now also J1.6 (Pin_6)
- net at Encoder1.3 (Pin_3): now also J1.8 (Pin_8)
- no-connect marks 0 -> 1

Commit message: chc
Connections:
- net +5V: now also J1.1 (Pin_1), J1.2 (Pin_2); no longer J1.11 (Pin_11), J1.12 (Pin_12)
- net GND: now also J1.11 (Pin_11), J1.12 (Pin_12); no longer J1.1 (Pin_1), J1.2 (Pin_2)
- net at R7.1, SW2.2: now also J1.8 (Pin_8); no longer J1.7 (Pin_7)
- net at J1.10 (Pin_10): now also R8.1, SW1.2
- net at R5.1, SW4.2: now also J1.4 (Pin_4); no longer J1.3 (Pin_3)
- net at Encoder1.1 (Pin_1): now also J1.5 (Pin_5); no longer J1.4 (Pin_4)
- net at R6.1, SW3.2: now also J1.6 (Pin_6); no longer J1.5 (Pin_5)
- net at Encoder1.2 (Pin_2): now also J1.7 (Pin_7); no longer J1.6 (Pin_6)
- net at Encoder1.3 (Pin_3): now also J1.9 (Pin_9); no longer J1.8 (Pin_8)
Other:
- moved on the sheet: Encoder1, R5, R6, R7, R8
