File: Proyecto Final/Circuitos del kicad/Placas/Main y ESP test socket/Placa_main_ESPtestsocket.kicad_sch (KiCad schematic)
At the start: 21 parts, among them J1 12v, J2 Conn_02x05_Odd_Even, J3 Conn_02x06_Odd_Even, J4 Conn_01x08, J5 Conn_01x08, J6 Conn_01x06, U1 LM7805, U2 ESP-12E, U3 ATmega328P-P, U4 LM1117-3.3, U5 BOB-12009, Y1 16MHz

Commit message: Agregado placa con zocalo piola
Parts:
- C1, C2, C3, C4, C5: footprint Capacitor_THT:C_Disc_D5.0mm_W2.5mm_P5.00mm -> Capacitor_THT:C_Disc_D5.0mm_W2.5mm_P2.50mm
- R1: footprint Resistor_THT:R_Axial_DIN0204_L3.6mm_D1.6mm_P5.08mm_Horizontal -> Resistor_THT:R_Axial_DIN0207_L6.3mm_D2.5mm_P7.62mm_Horizontal
- R2: footprint Resistor_THT:R_Axial_DIN0204_L3.6mm_D1.6mm_P5.08mm_Horizontal -> Resistor_THT:R_Axial_DIN0204_L3.6mm_D1.6mm_P1.90mm_Vertical
- U3: footprint Package_DIP:DIP-28_W7.62mm_LongPads -> Zocalo de fuerza:Zocalo_fuerza_40
Changed lines of the file:
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@@
       (effects (font (size 1.27 1.27)) (justify left))
     )
-    (property "Footprint" "Resistor_THT:R_Axial_DIN0204_L3.6mm_D1.6mm_P5.08mm_Horizontal" (id 2) (at 60.198 69.342 0)
+    (property "Footprint" "Resistor_THT:R_Axial_DIN0204_L3.6mm_D1.6mm_P1.90mm_Vertical" (id 2) (at 60.198 69.342 0)
       (effects (font (size 1.27 1.27)) hide)
     )
@@
     (property "Reference" "C2" (id 0) (at 90.424 44.1706 90))
     (property "Value" "20pF" (id 1) (at 90.424 46.7106 90))
-    (property "Footprint" "Capacitor_THT:C_Disc_D5.0mm_W2.5mm_P5.00mm" (id 2) (at 94.234 50.0888 0)
+    (property "Footprint" "Capacitor_THT:C_Disc_D5.0mm_W2.5mm_P2.50mm" (id 2) (at 94.234 50.0888 0)
       (effects (font (size 1.27 1.27)) hide)
     )
@@
       (effects (font (size 1.27 1.27)) (justify left))
     )
-    (property "Footprint" "Capacitor_THT:C_Disc_D5.0mm_W2.5mm_P5.00mm" (id 2) (at 84.1502 125.095 0)
+    (property "Footprint" "Capacitor_THT:C_Disc_D5.0mm_W2.5mm_P2.50mm" (id 2) (at 84.1502 125.095 0)
       (effects (font (size 1.27 1.27)) hide)
     )
@@
       (effects (font (size 1.27 1.27)) (justify left))
     )
-    (property "Footprint" "Resistor_THT:R_Axial_DIN0204_L3.6mm_D1.6mm_P5.08mm_Horizontal" (id 2) (at 124.968 24.892 0)
+    (property "Footprint" "Resistor_THT:R_Axial_DIN0207_L6.3mm_D2.5mm_P7.62mm_Horizontal" (id 2) (at 124.968 24.892 0)
       (effects (font (size 1.27 1.27)) hide)
     )
@@
     (property "Reference" "C1" (id 0) (at 90.17 27.5082 90))
     (property "Value" "20pF" (id 1) (at 90.17 30.0482 90))
-    (property "Footprint" "Capacitor_THT:C_Disc_D5.0mm_W2.5mm_P5.00mm" (id 2) (at 93.98 33.3248 0)
+    (property "Footprint" "Capacitor_THT:C_Disc_D5.0mm_W2.5mm_P2.50mm" (id 2) (at 93.98 33.3248 0)
       (effects (font (size 1.27 1.27)) hide)
     )
@@
       (effects (font (size 1.27 1.27)) (justify right))
     )
-    (property "Footprint" "Capacitor_THT:C_Disc_D5.0mm_W2.5mm_P5.00mm" (id 2) (at 210.6168 42.418 0)
+    (property "Footprint" "Capacitor_THT:C_Disc_D5.0mm_W2.5mm_P2.50mm" (id 2) (at 210.6168 42.418 0)
       (effects (font (size 1.27 1.27)) hide)
     )
@@
     )
     (property "Value" "ATmega328P-P" (id 1) (at 33.401 21.717 0))
-    (property "Footprint" "Package_DIP:DIP-28_W7.62mm_LongPads" (id 2) (at 42.418 61.722 0)
+    (property "Footprint" "Zocalo de fuerza:Zocalo_fuerza_40" (id 2) (at 42.418 61.722 0)
       (effects (font (size 1.27 1.27) italic) hide)
     )
@@
       (effects (font (size 1.27 1.27)) (justify right))
     )
-    (property "Footprint" "Capacitor_THT:C_Disc_D5.0mm_W2.5mm_P5.00mm" (id 2) (at 230.9368 42.418 0)
+    (property "Footprint" "Capacitor_THT:C_Disc_D5.0mm_W2.5mm_P2.50mm" (id 2) (at 230.9368 42.418 0)
       (effects (font (size 1.27 1.27)) hide)
     )
@@
     )
     (path "/9a83f868-a35b-409e-b071-e3aadc30670b"
-      (reference "C1") (unit 1) (value "20pF") (footprint "Capacitor_THT:C_Disc_D5.0mm_W2.5mm_P5.00mm")
+      (reference "C1") (unit 1) (value "20pF") (footprint "Capacitor_THT:C_Disc_D5.0mm_W2.5mm_P2.50mm")
     )
     (path "/51abec91-c28a-444c-9af7-82393bd86496"
-      (reference "C2") (unit 1) (value "20pF") (footprint "Capacitor_THT:C_Disc_D5.0mm_W2.5mm_P5.00mm")
+      (reference "C2") (unit 1) (value "20pF") (footprint "Capacitor_THT:C_Disc_D5.0mm_W2.5mm_P2.50mm")
     )
     (path "/abbe8f28-5a3c-493c-bd33-e8f3c31b566d"
-      (reference "C3") (unit 1) (value "330nF") (footprint "Capacitor_THT:C_Disc_D5.0mm_W2.5mm_P5.00mm")
+      (reference "C3") (unit 1) (value "330nF") (footprint "Capacitor_THT:C_Disc_D5.0mm_W2.5mm_P2.50mm")
     )
     (path "/e07aa1df-61c5-4103-8f65-c85706f29286"
-      (reference "C4") (unit 1) (value "100nF") (footprint "Capacitor_THT:C_Disc_D5.0mm_W2.5mm_P5.00mm")
+      (reference "C4") (unit 1) (value "100nF") (footprint "Capacitor_THT:C_Disc_D5.0mm_W2.5mm_P2.50mm")
     )
     (path "/69027843-a488-48d6-b151-31c8144d0709"
-      (reference "C5") (unit 1) (value "100nF") (footprint "Capacitor_THT:C_Disc_D5.0mm_W2.5mm_P5.00mm")
+      (reference "C5") (unit 1) (value "100nF") (footprint "Capacitor_THT:C_Disc_D5.0mm_W2.5mm_P2.50mm")
     )
     (path "/d2fe5be2-0af9-4b0e-af75-c9dd79dbc3d5"
@@
     )
     (path "/6a730b26-141b-4550-bfbd-6131095893ab"
-      (reference "R1") (unit 1) (value "4.7k") (footprint "Resistor_THT:R_Axial_DIN0204_L3.6mm_D1.6mm_P5.08mm_Horizontal")
+      (reference "R1") (unit 1) (value "4.7k") (footprint "Resistor_THT:R_Axial_DIN0207_L6.3mm_D2.5mm_P7.62mm_Horizontal")
     )
     (path "/2503c218-3d1f-4043-8942-c69a3519b522"
-      (reference "R2") (unit 1) (value "10k") (footprint "Resistor_THT:R_Axial_DIN0204_L3.6mm_D1.6mm_P5.08mm_Horizontal")
+      (reference "R2") (unit 1) (value "10k") (footprint "Resistor_THT:R_Axial_DIN0204_L3.6mm_D1.6mm_P1.90mm_Vertical")
     )
     (path "/235eb236-c253-4810-915e-7bfdbb88a9cf"
@@
     )
     (path "/b6baee3f-9d6c-4256-afdd-f7ec59c8a6a2"
-      (reference "U3") (unit 1) (value "ATmega328P-P") (footprint "Package_DIP:DIP-28_W7.62mm_LongPads")
+      (reference "U3") (unit 1) (value "ATmega328P-P") (footprint "Zocalo de fuerza:Zocalo_fuerza_40")
     )
     (path "/fef04073-b9b3-42d1-91c5-248a55a47691"
