File: Proyecto Final/Circuitos del kicad/Placas/Main y ESP test socket/Placa_main_ESPtestsocket.kicad_pcb (KiCad board)
At the start: 2 copper layers, 86.1 x 113.3 mm, 17 parts, among them J1 12v, J2 Conn_02x05_Odd_Even, J3 Conn_02x06_Odd_Even, U1 LM7805, U3 ATmega328P-P, U4 LM1117-3.3, U5 BOB-12009, Y1 16MHz

Commit message: Cambio layout placa main
Parts:
- moved J1 52.2 mm to (100.1, 123.9), turned to -90 degrees
- moved C3 43.6 mm to (106.2, 126.5), turned to -90 degrees
- moved U1 31.9 mm to (114.8, 129.0), turned to 90 degrees
- moved C4 20.2 mm to (123.2, 121.7), turned to -90 degrees
Routing:
- net Net-(J3-Pad7): track 223.6 -> 194.2 mm
- net GND: track 371.7 -> 396.2 mm
- net +12V: track 78.0 -> 91.7 mm
Other:
- board size 86.1 x 113.3 mm -> 86.1 x 88.2 mm

Commit message: wewew
Parts:
- moved C5 6.10 mm to (143.8, 64.0)
- moved R1 0.51 mm to (158.5, 88.6)
Routing:
- net +5V: track 292.6 -> 299.7 mm
- net GND: track 396.2 -> 391.2 mm
- net Net-(J3-Pad10): track 34.9 -> 31.2 mm
- net Net-(J3-Pad8): track 36.3 -> 32.6 mm
- net Net-(J3-Pad6): track 36.8 -> 33.1 mm
- net Net-(C6-Pad1): track 55.7 -> 59.0 mm
- net Net-(J2-Pad8): track 40.0 -> 39.5 mm
Other:
- board text added: "3.3v"
- board text added: "5v"
- board text added: "RX"
- board text added: "TX"
- board text removed: "+"
