File: Proyecto Final/Circuitos del kicad/Placas/Placa relays/Placa_relays.kicad_pcb (KiCad board)
At the start: 2 copper layers, 89.9 x 85.7 mm, 23 parts, among them J1 Conn_02x05_Odd_Even, Q1 PN2222A, Q2 PN2222A, Q3 PN2222A

Commit message: wewew
Parts:
- R1, R5, R6: footprint Resistor_THT:R_Axial_DIN0204_L3.6mm_D1.6mm_P5.08mm_Horizontal -> Resistor_THT:R_Axial_DIN0207_L6.3mm_D2.5mm_P7.62mm_Horizontal
- R2, R3, R4: footprint Resistor_THT:R_Axial_DIN0204_L3.6mm_D1.6mm_P7.62mm_Horizontal -> Resistor_THT:R_Axial_DIN0207_L6.3mm_D2.5mm_P7.62mm_Horizontal
- moved R5 1.59 mm to (135.6, 91.5)
- moved R1 1.41 mm to (133.6, 109.2)
- moved R2 1.37 mm to (126.0, 96.5)
- moved R6 0.17 mm to (137.4, 72.4)
Routing:
- net +12V: track 182.8 -> 185.7 mm
- net Net-(Q3-Pad2): track 25.5 -> 22.8 mm
- net Net-(Q2-Pad2): track 20.3 -> 18.7 mm
- net Net-(J1-Pad8): track 10.6 -> 11.9 mm
- net Net-(D5-Pad2): track 4.87 -> 3.81 mm
- net Net-(D6-Pad2): track 8.42 -> 9.35 mm
- net Net-(D4-Pad2): track 13.2 -> 12.5 mm
